Commit message: Completed simulation environment setup

File: assets/urdf/AR5_L6_description/AR5_L6_right.urdf (robot description, URDF)
Before this commit: robot AR5_L6_right, 27 links, 26 joints
Links:
- removed link AR5-5_07R-W4C4A2_base
- removed link AR5-5_07R-W4C4A2_link1
- removed link AR5-5_07R-W4C4A2_link2
- removed link AR5-5_07R-W4C4A2_link3
- removed link AR5-5_07R-W4C4A2_link4
- removed link AR5-5_07R-W4C4A2_link5
- removed link AR5-5_07R-W4C4A2_link6
- removed link AR5-5_07R-W4C4A2_link7
- removed link AR5-5_07R-W4C4A2_tcp
- added link AR5_5_07R_W4C4A2_base; collision mesh filename=AR5_right_meshes/AR5_5_07R_W4C4A2_base.stl scale=0.001 0.001 0.001; visual mesh filename=AR5_right_meshes/AR5_5_07R_W4C4A2_base.stl scale=0.001 0.001 0.001
- added link AR5_5_07R_W4C4A2_link1, mass 2.683; collision mesh filename=AR5_right_meshes/AR5_5_07R_W4C4A2_link1.stl scale=0.001 0.001 0.001; visual mesh filename=AR5_right_meshes/AR5_5_07R_W4C4A2_link1.stl scale=0.001 0.001 0.001
- added link AR5_5_07R_W4C4A2_link2, mass 2.3; collision mesh filename=AR5_right_meshes/AR5_5_07R_W4C4A2_link2.stl scale=0.001 0.001 0.001; visual mesh filename=AR5_right_meshes/AR5_5_07R_W4C4A2_link2.stl scale=0.001 0.001 0.001
- added link AR5_5_07R_W4C4A2_link3, mass 1.862; collision mesh filename=AR5_right_meshes/AR5_5_07R_W4C4A2_link3.stl scale=0.001 0.001 0.001; visual mesh filename=AR5_right_meshes/AR5_5_07R_W4C4A2_link3.stl scale=0.001 0.001 0.001
- added link AR5_5_07R_W4C4A2_link4, mass 1.234; collision mesh filename=AR5_right_meshes/AR5_5_07R_W4C4A2_link4.stl scale=0.001 0.001 0.001; visual mesh filename=AR5_right_meshes/AR5_5_07R_W4C4A2_link4.stl scale=0.001 0.001 0.001
- added link AR5_5_07R_W4C4A2_link5, mass 1.328; collision mesh filename=AR5_right_meshes/AR5_5_07R_W4C4A2_link5.stl scale=0.001 0.001 0.001; visual mesh filename=AR5_right_meshes/AR5_5_07R_W4C4A2_link5.stl scale=0.001 0.001 0.001
- added link AR5_5_07R_W4C4A2_link6, mass 0.93; collision mesh filename=AR5_right_meshes/AR5_5_07R_W4C4A2_link6.stl scale=0.001 0.001 0.001; visual mesh filename=AR5_right_meshes/AR5_5_07R_W4C4A2_link6.stl scale=0.001 0.001 0.001
- added link AR5_5_07R_W4C4A2_link7, mass 0.332; collision mesh filename=AR5_right_meshes/AR5_5_07R_W4C4A2_link7.stl scale=0.001 0.001 0.001; visual mesh filename=AR5_right_meshes/AR5_5_07R_W4C4A2_link7.stl scale=0.001 0.001 0.001
- added link AR5_5_07R_W4C4A2_tcp, mass 0.0; collision box size=0.0001 0.0001 0.0001; visual box size=0.0001 0.0001 0.0001
- link rh_index_tip: geometry collision box size=0.0001 0.0001 0.0001; visual box size=0.0001 0.0001 0.0001
- link rh_middle_tip: geometry collision box size=0.0001 0.0001 0.0001; visual box size=0.0001 0.0001 0.0001
- link rh_pinky_tip: geometry collision box size=0.0001 0.0001 0.0001; visual box size=0.0001 0.0001 0.0001
- link rh_ring_tip: geometry collision box size=0.0001 0.0001 0.0001; visual box size=0.0001 0.0001 0.0001
- link rh_thumb_tip: geometry collision box size=0.0001 0.0001 0.0001; visual box size=0.0001 0.0001 0.0001
- link world: geometry collision box size=0.0001 0.0001 0.0001; visual box size=0.0001 0.0001 0.0001
Joints:
- removed joint AR5-5_07R-W4C4A2_joint_1
- removed joint AR5-5_07R-W4C4A2_joint_2
- removed joint AR5-5_07R-W4C4A2_joint_3
- removed joint AR5-5_07R-W4C4A2_joint_4
- removed joint AR5-5_07R-W4C4A2_joint_5
- removed joint AR5-5_07R-W4C4A2_joint_6
- removed joint AR5-5_07R-W4C4A2_joint_7
- removed joint AR5-5_07R-W4C4A2_tcp_joint
- added joint AR5_5_07R_W4C4A2_joint_1: type revolute, parent AR5_5_07R_W4C4A2_base, child AR5_5_07R_W4C4A2_link1, origin xyz=0.0 0.0 0.0 rpy=0 0 0, axis 0 0 1, limit lower=-3.1067 upper=3.1067 effort=108 velocity=3.0543261909900763
- added joint AR5_5_07R_W4C4A2_joint_2: type revolute, parent AR5_5_07R_W4C4A2_link1, child AR5_5_07R_W4C4A2_link2, origin xyz=0.0 0.0 0.1745 rpy=0 0 0, axis 0 1 0, limit lower=-2.0944 upper=2.0944 effort=108 velocity=3.0543261909900763
- added joint AR5_5_07R_W4C4A2_joint_3: type revolute, parent AR5_5_07R_W4C4A2_link2, child AR5_5_07R_W4C4A2_link3, origin xyz=0.0 0.0 0.314 rpy=0 0 0, axis 0 0 1, limit lower=-3.1067 upper=3.1067 effort=66 velocity=4.71238898038469
- added joint AR5_5_07R_W4C4A2_joint_4: type revolute, parent AR5_5_07R_W4C4A2_link3, child AR5_5_07R_W4C4A2_link4, origin xyz=0.01 0.0 0.0 rpy=0 0 0, axis 0 1 0, limit lower=-1.0472 upper=2.5307 effort=66 velocity=5.235987755982989
- added joint AR5_5_07R_W4C4A2_joint_5: type revolute, parent AR5_5_07R_W4C4A2_link4, child AR5_5_07R_W4C4A2_link5, origin xyz=-0.01 0.0 0.272 rpy=0 0 0, axis 0 0 1, limit lower=-3.1067 upper=3.1067 effort=19 velocity=4.1887902047863905
- added joint AR5_5_07R_W4C4A2_joint_6: type revolute, parent AR5_5_07R_W4C4A2_link5, child AR5_5_07R_W4C4A2_link6, origin xyz=0.0 0.0 0.0 rpy=0.0 0.0 0, axis 0 1 0, limit lower=-1.0472 upper=1.0472 effort=19 velocity=4.1887902047863905
- added joint AR5_5_07R_W4C4A2_joint_7: type revolute, parent AR5_5_07R_W4C4A2_link6, child AR5_5_07R_W4C4A2_link7, origin xyz=0.0 0.0 0.0 rpy=0.0 0.0 0, axis 1 0 0, limit lower=-1.0472 upper=1.0472 effort=19 velocity=4.1887902047863905
- added joint AR5_5_07R_W4C4A2_tcp_joint: type fixed, parent AR5_5_07R_W4C4A2_link7, child AR5_5_07R_W4C4A2_tcp, origin xyz=0.0 0.0 0.097 rpy=0 0 0
- joint arm_hand_fixed: parent AR5-5_07R-W4C4A2_tcp -> AR5_5_07R_W4C4A2_tcp
- joint fixed: child AR5-5_07R-W4C4A2_base -> AR5_5_07R_W4C4A2_base

File: assets/urdf/AR5_L6_description/archive/AR5_L6_right_workstation.urdf (robot description, URDF)
Before this commit: robot AR5_L6_left, 27 links, 26 joints
Links:
- removed link AR5_5_07L_W4C4A2_base
- removed link AR5_5_07L_W4C4A2_link1
- removed link AR5_5_07L_W4C4A2_link2
- removed link AR5_5_07L_W4C4A2_link3
- removed link AR5_5_07L_W4C4A2_link4
- removed link AR5_5_07L_W4C4A2_link5
- removed link AR5_5_07L_W4C4A2_link6
- removed link AR5_5_07L_W4C4A2_link7
- removed link AR5_5_07L_W4C4A2_tcp
- removed link lh_hand_base_link
- removed link lh_index_distal
- removed link lh_index_proximal
- removed link lh_index_tip
- removed link lh_middle_distal
- removed link lh_middle_proximal
- removed link lh_middle_tip
- removed link lh_pinky_distal
- removed link lh_pinky_proximal
- removed link lh_pinky_tip
- removed link lh_ring_distal
- removed link lh_ring_proximal
- removed link lh_ring_tip
- removed link lh_thumb_distal
- removed link lh_thumb_metacarpals
- removed link lh_thumb_metacarpals_base1
- removed link lh_thumb_tip
- added link AR5_5_07R_W4C4A2_base; collision mesh filename=AR5_right_meshes/AR5_5_07R_W4C4A2_base.stl scale=0.001 0.001 0.001; visual mesh filename=AR5_right_meshes/AR5_5_07R_W4C4A2_base.stl scale=0.001 0.001 0.001
- added link AR5_5_07R_W4C4A2_link1, mass 2.683; collision mesh filename=AR5_right_meshes/AR5_5_07R_W4C4A2_link1.stl scale=0.001 0.001 0.001; visual mesh filename=AR5_right_meshes/AR5_5_07R_W4C4A2_link1.stl scale=0.001 0.001 0.001
- added link AR5_5_07R_W4C4A2_link2, mass 2.3; collision mesh filename=AR5_right_meshes/AR5_5_07R_W4C4A2_link2.stl scale=0.001 0.001 0.001; visual mesh filename=AR5_right_meshes/AR5_5_07R_W4C4A2_link2.stl scale=0.001 0.001 0.001
- added link AR5_5_07R_W4C4A2_link3, mass 1.862; collision mesh filename=AR5_right_meshes/AR5_5_07R_W4C4A2_link3.stl scale=0.001 0.001 0.001; visual mesh filename=AR5_right_meshes/AR5_5_07R_W4C4A2_link3.stl scale=0.001 0.001 0.001
- added link AR5_5_07R_W4C4A2_link4, mass 1.234; collision mesh filename=AR5_right_meshes/AR5_5_07R_W4C4A2_link4.stl scale=0.001 0.001 0.001; visual mesh filename=AR5_right_meshes/AR5_5_07R_W4C4A2_link4.stl scale=0.001 0.001 0.001
- added link AR5_5_07R_W4C4A2_link5, mass 1.328; collision mesh filename=AR5_right_meshes/AR5_5_07R_W4C4A2_link5.stl scale=0.001 0.001 0.001; visual mesh filename=AR5_right_meshes/AR5_5_07R_W4C4A2_link5.stl scale=0.001 0.001 0.001
- added link AR5_5_07R_W4C4A2_link6, mass 0.93; collision mesh filename=AR5_right_meshes/AR5_5_07R_W4C4A2_link6.stl scale=0.001 0.001 0.001; visual mesh filename=AR5_right_meshes/AR5_5_07R_W4C4A2_link6.stl scale=0.001 0.001 0.001
- added link AR5_5_07R_W4C4A2_link7, mass 0.332; collision mesh filename=AR5_right_meshes/AR5_5_07R_W4C4A2_link7.stl scale=0.001 0.001 0.001; visual mesh filename=AR5_right_meshes/AR5_5_07R_W4C4A2_link7.stl scale=0.001 0.001 0.001
- added link AR5_5_07R_W4C4A2_tcp, mass 0.0; collision box size=0.0001 0.0001 0.0001; visual box size=0.0001 0.0001 0.0001
- added link rh_hand_base_link, mass 0.4185; collision mesh filename=L6_right_meshes/hand_base_link.STL; visual mesh filename=L6_right_meshes/hand_base_link.STL
- added link rh_index_distal, mass 0.018408; collision mesh filename=L6_right_meshes/index_distal.STL; visual mesh filename=L6_right_meshes/index_distal.STL
- added link rh_index_proximal, mass 0.008553; collision mesh filename=L6_right_meshes/index_proximal.STL; visual mesh filename=L6_right_meshes/index_proximal.STL
- added link rh_index_tip, mass 1e-06; collision box size=0.0001 0.0001 0.0001; visual box size=0.0001 0.0001 0.0001
- added link rh_middle_distal, mass 0.018408; collision mesh filename=L6_right_meshes/middle_distal.STL; visual mesh filename=L6_right_meshes/middle_distal.STL
- added link rh_middle_proximal, mass 0.008553; collision mesh filename=L6_right_meshes/middle_proximal.STL; visual mesh filename=L6_right_meshes/middle_proximal.STL
- added link rh_middle_tip, mass 1e-06; collision box size=0.0001 0.0001 0.0001; visual box size=0.0001 0.0001 0.0001
- added link rh_pinky_distal, mass 0.018408; collision mesh filename=L6_right_meshes/pinky_distal.STL; visual mesh filename=L6_right_meshes/pinky_distal.STL
- added link rh_pinky_proximal, mass 0.008553; collision mesh filename=L6_right_meshes/pinky_proximal.STL; visual mesh filename=L6_right_meshes/pinky_proximal.STL
- added link rh_pinky_tip, mass 1e-06; collision box size=0.0001 0.0001 0.0001; visual box size=0.0001 0.0001 0.0001
- added link rh_ring_distal, mass 0.018408; collision mesh filename=L6_right_meshes/ring_distal.STL; visual mesh filename=L6_right_meshes/ring_distal.STL
- added link rh_ring_proximal, mass 0.008553; collision mesh filename=L6_right_meshes/ring_proximal.STL; visual mesh filename=L6_right_meshes/ring_proximal.STL
- added link rh_ring_tip, mass 1e-06; collision box size=0.0001 0.0001 0.0001; visual box size=0.0001 0.0001 0.0001
- added link rh_thumb_distal, mass 0.018; collision mesh filename=L6_right_meshes/thumb_distal.STL; visual mesh filename=L6_right_meshes/thumb_distal.STL
- added link rh_thumb_metacarpals, mass 0.065; collision mesh filename=L6_right_meshes/thumb_metacarpals.STL; visual mesh filename=L6_right_meshes/thumb_metacarpals.STL
- added link rh_thumb_metacarpals_base1, mass 0.01; collision mesh filename=L6_right_meshes/thumb_metacarpals_base1.STL; visual mesh filename=L6_right_meshes/thumb_metacarpals_base1.STL
- added link rh_thumb_tip, mass 1e-06; collision box size=0.0001 0.0001 0.0001; visual box size=0.0001 0.0001 0.0001
- added link workstation_link, mass 50.0; collision mesh filename=../workstation.STL; visual mesh filename=../workstation.STL
- link world: geometry 
Joints:
- removed joint AR5_5_07L_W4C4A2_joint_1
- removed joint AR5_5_07L_W4C4A2_joint_2
- removed joint AR5_5_07L_W4C4A2_joint_3
- removed joint AR5_5_07L_W4C4A2_joint_4
- removed joint AR5_5_07L_W4C4A2_joint_5
- removed joint AR5_5_07L_W4C4A2_joint_6
- removed joint AR5_5_07L_W4C4A2_joint_7
- removed joint AR5_5_07L_W4C4A2_tcp_joint
- removed joint fixed
- removed joint lh_index_dip
- removed joint lh_index_mcp_pitch
- removed joint lh_index_tip_fixed
- removed joint lh_middle_dip
- removed joint lh_middle_mcp_pitch
- removed joint lh_middle_tip_fixed
- removed joint lh_pinky_dip
- removed joint lh_pinky_mcp_pitch
- removed joint lh_pinky_tip_fixed
- removed joint lh_ring_dip
- removed joint lh_ring_mcp_pitch
- removed joint lh_ring_tip_fixed
- removed joint lh_thumb_cmc_pitch
- removed joint lh_thumb_cmc_roll
- removed joint lh_thumb_dip
- removed joint lh_thumb_tip_fixed
- added joint AR5_5_07R_W4C4A2_joint_1: type revolute, parent AR5_5_07R_W4C4A2_base, child AR5_5_07R_W4C4A2_link1, origin xyz=0.0 0.0 0.0 rpy=0 0 0, axis 0 0 1, limit lower=-3.1067 upper=3.1067 effort=108 velocity=3.0543261909900763
- added joint AR5_5_07R_W4C4A2_joint_2: type revolute, parent AR5_5_07R_W4C4A2_link1, child AR5_5_07R_W4C4A2_link2, origin xyz=0.0 0.0 0.1745 rpy=0 0 0, axis 0 1 0, limit lower=-2.0944 upper=2.0944 effort=108 velocity=3.0543261909900763
- added joint AR5_5_07R_W4C4A2_joint_3: type revolute, parent AR5_5_07R_W4C4A2_link2, child AR5_5_07R_W4C4A2_link3, origin xyz=0.0 0.0 0.314 rpy=0 0 0, axis 0 0 1, limit lower=-3.1067 upper=3.1067 effort=66 velocity=4.71238898038469
- added joint AR5_5_07R_W4C4A2_joint_4: type revolute, parent AR5_5_07R_W4C4A2_link3, child AR5_5_07R_W4C4A2_link4, origin xyz=0.01 0.0 0.0 rpy=0 0 0, axis 0 1 0, limit lower=-1.0472 upper=2.5307 effort=66 velocity=5.235987755982989
- added joint AR5_5_07R_W4C4A2_joint_5: type revolute, parent AR5_5_07R_W4C4A2_link4, child AR5_5_07R_W4C4A2_link5, origin xyz=-0.01 0.0 0.272 rpy=0 0 0, axis 0 0 1, limit lower=-3.1067 upper=3.1067 effort=19 velocity=4.1887902047863905
- added joint AR5_5_07R_W4C4A2_joint_6: type revolute, parent AR5_5_07R_W4C4A2_link5, child AR5_5_07R_W4C4A2_link6, origin xyz=0.0 0.0 0.0 rpy=0.0 0.0 0, axis 0 1 0, limit lower=-1.0472 upper=1.0472 effort=19 velocity=4.1887902047863905
- added joint AR5_5_07R_W4C4A2_joint_7: type revolute, parent AR5_5_07R_W4C4A2_link6, child AR5_5_07R_W4C4A2_link7, origin xyz=0.0 0.0 0.0 rpy=0.0 0.0 0, axis 1 0 0, limit lower=-1.0472 upper=1.0472 effort=19 velocity=4.1887902047863905
- added joint AR5_5_07R_W4C4A2_tcp_joint: type fixed, parent AR5_5_07R_W4C4A2_link7, child AR5_5_07R_W4C4A2_tcp, origin xyz=0.0 0.0 0.097 rpy=0 0 0
- added joint rh_index_dip: type revolute, parent rh_index_proximal, child rh_index_distal, origin xyz=0.0009359 0 0.028002 rpy=0 0 0, axis 0 1 0, limit lower=0 upper=1.277039 effort=0 velocity=3.1, mimic joint=rh_index_mcp_pitch multiplier=1.125676 offset=0
- added joint rh_index_mcp_pitch: type revolute, parent rh_hand_base_link, child rh_index_proximal, origin xyz=-0.00066821 0.033467 0.11622 rpy=-0.087266 0 0, axis 0 1 0, limit lower=0 upper=1.134464 effort=0.574 velocity=6.10
- added joint rh_index_tip_fixed: type fixed, parent rh_index_distal, child rh_index_tip, origin xyz=0.0341 0 0.034 rpy=0 0 0
- added joint rh_middle_dip: type revolute, parent rh_middle_proximal, child rh_middle_distal, origin xyz=0.0009359 0 0.028002 rpy=0 0 0, axis 0 1 0, limit lower=0 upper=1.277039 effort=0 velocity=3.1, mimic joint=rh_middle_mcp_pitch multiplier=1.125676 offset=0
- added joint rh_middle_mcp_pitch: type revolute, parent rh_hand_base_link, child rh_middle_proximal, origin xyz=-0.00066821 0.0134013 0.12272 rpy=-0.034907 0 0, axis 0 1 0, limit lower=0 upper=1.134464 effort=0.574 velocity=6.10
- added joint rh_middle_tip_fixed: type fixed, parent rh_middle_distal, child rh_middle_tip, origin xyz=0.0341 0 0.034 rpy=0 0 0
- added joint rh_pinky_dip: type revolute, parent rh_pinky_proximal, child rh_pinky_distal, origin xyz=0.0009359 0 0.028002 rpy=0 0 0, axis 0 1 0, limit lower=0 upper=1.277039 effort=0 velocity=3.1, mimic joint=rh_pinky_mcp_pitch multiplier=1.125676 offset=0
- added joint rh_pinky_mcp_pitch: type revolute, parent rh_hand_base_link, child rh_pinky_proximal, origin xyz=-0.00067852 -0.025314 0.11474 rpy=0.05236 0 0, axis 0 1 0, limit lower=0 upper=1.134464 effort=0.574 velocity=6.10
- added joint rh_pinky_tip_fixed: type fixed, parent rh_pinky_distal, child rh_pinky_tip, origin xyz=0.0341 0 0.034 rpy=0 0 0
- added joint rh_ring_dip: type revolute, parent rh_ring_proximal, child rh_ring_distal, origin xyz=0.0009359 0 0.028002 rpy=0 0 0, axis 0 1 0, limit lower=0 upper=1.277039 effort=0 velocity=3.1, mimic joint=rh_ring_mcp_pitch multiplier=1.125676 offset=0
- added joint rh_ring_mcp_pitch: type revolute, parent rh_hand_base_link, child rh_ring_proximal, origin xyz=-0.00067368 -0.006217 0.11872 rpy=0.017453 0 0, axis 0 1 0, limit lower=0 upper=1.134464 effort=0.574 velocity=6.10
- added joint rh_ring_tip_fixed: type fixed, parent rh_ring_distal, child rh_ring_tip, origin xyz=0.0341 0 0.034 rpy=0 0 0
- added joint rh_thumb_cmc_pitch: type revolute, parent rh_thumb_metacarpals_base1, child rh_thumb_metacarpals, origin xyz=0.0054997 0.013314 0.0032166 rpy=-1.0762 0.013637 -0.40121, axis 1 0 0, limit lower=0 upper=0.837758 effort=1.008 velocity=3.47
- added joint rh_thumb_cmc_roll: type revolute, parent rh_hand_base_link, child rh_thumb_metacarpals_base1, origin xyz=0.0078133 0.030812 0.025678 rpy=-0.034907 0 0, axis 0 0.034899 -0.99939, limit lower=-0.087266 upper=1.256637 effort=0.588 velocity=5.95
- added joint rh_thumb_dip: type revolute, parent rh_thumb_metacarpals, child rh_thumb_distal, origin xyz=0 -0.0061 0.0827 rpy=0 0 0, axis 1 0 0, limit lower=0 upper=0.963287 effort=0 velocity=1.7, mimic joint=rh_thumb_cmc_pitch multiplier=1.226495 offset=0
- added joint rh_thumb_tip_fixed: type fixed, parent rh_thumb_distal, child rh_thumb_tip, origin xyz=0 -0.0035 0.026 rpy=0 0 -1.5708
- added joint workstation_to_arm_base: type fixed, parent workstation_link, child AR5_5_07R_W4C4A2_base, origin xyz=0.0637 0.536 1.267 rpy=1.5708 1.5708 0
- added joint world_to_workstation: type fixed, parent world, child workstation_link, origin xyz=0 0 0 rpy=0 0 0
- joint arm_hand_fixed: child lh_hand_base_link -> rh_hand_base_link; origin xyz=0 0 0.03 rpy=0 0 1.5708 -> xyz=0 0 0.03 rpy=0 0 -1.5708; parent AR5_5_07L_W4C4A2_tcp -> AR5_5_07R_W4C4A2_tcp
