Commit message: Added functionality tests for ppo pipeline (#1)
Modified and integrated URDF. Setup controller tuning pipeline.

---------

Co-authored-by: Ryan Zhou <ryanzed12138@gmail.com>
Reviewed-on: https://gitea.linkerhub.work/zhouhaoyu/dex-tool-rl/pulls/1

File: assets/urdf/AR5_L6_description/archive/L6_V3_1R/linkerhand_L6V3.1_right.urdf (robot description, URDF)
Before this commit: robot linkerhand_L6V3.1_left_2.2, 17 links, 16 joints
Links:
- removed link lh_hand_base_link
- removed link lh_index_distal
- removed link lh_index_proximal
- removed link lh_index_tip
- removed link lh_middle_distal
- removed link lh_middle_proximal
- removed link lh_middle_tip
- removed link lh_pinky_distal
- removed link lh_pinky_proximal
- removed link lh_pinky_tip
- removed link lh_ring_distal
- removed link lh_ring_proximal
- removed link lh_ring_tip
- removed link lh_thumb_distal
- removed link lh_thumb_metacarpals
- removed link lh_thumb_metacarpals_base1
- removed link lh_thumb_tip
- added link rh_hand_base_link, mass 0.4185; collision mesh filename=../../L6_right_meshes/hand_base_link.STL; visual mesh filename=../../L6_right_meshes/hand_base_link.STL
- added link rh_index_distal, mass 0.018408; collision mesh filename=../../L6_right_meshes/index_distal.STL; visual mesh filename=../../L6_right_meshes/index_distal.STL
- added link rh_index_proximal, mass 0.008553; collision mesh filename=../../L6_right_meshes/index_proximal.STL; visual mesh filename=../../L6_right_meshes/index_proximal.STL
- added link rh_index_tip, mass 1e-06
- added link rh_middle_distal, mass 0.018408; collision mesh filename=../../L6_right_meshes/middle_distal.STL; visual mesh filename=../../L6_right_meshes/middle_distal.STL
- added link rh_middle_proximal, mass 0.008553; collision mesh filename=../../L6_right_meshes/middle_proximal.STL; visual mesh filename=../../L6_right_meshes/middle_proximal.STL
- added link rh_middle_tip, mass 1e-06
- added link rh_pinky_distal, mass 0.018408; collision mesh filename=../../L6_right_meshes/pinky_distal.STL; visual mesh filename=../../L6_right_meshes/pinky_distal.STL
- added link rh_pinky_proximal, mass 0.008553; collision mesh filename=../../L6_right_meshes/pinky_proximal.STL; visual mesh filename=../../L6_right_meshes/pinky_proximal.STL
- added link rh_pinky_tip, mass 1e-06
- added link rh_ring_distal, mass 0.018408; collision mesh filename=../../L6_right_meshes/ring_distal.STL; visual mesh filename=../../L6_right_meshes/ring_distal.STL
- added link rh_ring_proximal, mass 0.008553; collision mesh filename=../../L6_right_meshes/ring_proximal.STL; visual mesh filename=../../L6_right_meshes/ring_proximal.STL
- added link rh_ring_tip, mass 1e-06
- added link rh_thumb_distal, mass 0.018; collision mesh filename=../../L6_right_meshes/thumb_distal.STL; visual mesh filename=../../L6_right_meshes/thumb_distal.STL
- added link rh_thumb_metacarpals, mass 0.065; collision mesh filename=../../L6_right_meshes/thumb_metacarpals.STL; visual mesh filename=../../L6_right_meshes/thumb_metacarpals.STL
- added link rh_thumb_metacarpals_base1, mass 0.01; collision mesh filename=../../L6_right_meshes/thumb_metacarpals_base1.STL; visual mesh filename=../../L6_right_meshes/thumb_metacarpals_base1.STL
- added link rh_thumb_tip, mass 1e-06
Joints:
- removed joint lh_index_dip
- removed joint lh_index_mcp_pitch
- removed joint lh_index_tip_fixed
- removed joint lh_middle_dip
- removed joint lh_middle_mcp_pitch
- removed joint lh_middle_tip_fixed
- removed joint lh_pinky_dip
- removed joint lh_pinky_mcp_pitch
- removed joint lh_pinky_tip_fixed
- removed joint lh_ring_dip
- removed joint lh_ring_mcp_pitch
- removed joint lh_ring_tip_fixed
- removed joint lh_thumb_cmc_pitch
- removed joint lh_thumb_cmc_roll
- removed joint lh_thumb_dip
- removed joint lh_thumb_tip_fixed
- added joint rh_index_dip: type revolute, parent rh_index_proximal, child rh_index_distal, origin xyz=0.0009359 0 0.028002 rpy=0 0 0, axis 0 1 0, limit lower=0 upper=1.277039 effort=0 velocity=3.1, mimic joint=rh_index_mcp_pitch multiplier=1.125676 offset=0
- added joint rh_index_mcp_pitch: type revolute, parent rh_hand_base_link, child rh_index_proximal, origin xyz=-0.00066821 0.033467 0.11622 rpy=-0.087266 0 0, axis 0 1 0, limit lower=0 upper=1.134464 effort=0.574 velocity=6.10
- added joint rh_index_tip_fixed: type fixed, parent rh_index_distal, child rh_index_tip, origin xyz=0.0341 0 0.034 rpy=0 0 0
- added joint rh_middle_dip: type revolute, parent rh_middle_proximal, child rh_middle_distal, origin xyz=0.0009359 0 0.028002 rpy=0 0 0, axis 0 1 0, limit lower=0 upper=1.277039 effort=0 velocity=3.1, mimic joint=rh_middle_mcp_pitch multiplier=1.125676 offset=0
- added joint rh_middle_mcp_pitch: type revolute, parent rh_hand_base_link, child rh_middle_proximal, origin xyz=-0.00066821 0.0134013 0.12272 rpy=-0.034907 0 0, axis 0 1 0, limit lower=0 upper=1.134464 effort=0.574 velocity=6.10
- added joint rh_middle_tip_fixed: type fixed, parent rh_middle_distal, child rh_middle_tip, origin xyz=0.0341 0 0.034 rpy=0 0 0
- added joint rh_pinky_dip: type revolute, parent rh_pinky_proximal, child rh_pinky_distal, origin xyz=0.0009359 0 0.028002 rpy=0 0 0, axis 0 1 0, limit lower=0 upper=1.277039 effort=0 velocity=3.1, mimic joint=rh_pinky_mcp_pitch multiplier=1.125676 offset=0
- added joint rh_pinky_mcp_pitch: type revolute, parent rh_hand_base_link, child rh_pinky_proximal, origin xyz=-0.00067852 -0.025314 0.11474 rpy=0.05236 0 0, axis 0 1 0, limit lower=0 upper=1.134464 effort=0.574 velocity=6.10
- added joint rh_pinky_tip_fixed: type fixed, parent rh_pinky_distal, child rh_pinky_tip, origin xyz=0.0341 0 0.034 rpy=0 0 0
- added joint rh_ring_dip: type revolute, parent rh_ring_proximal, child rh_ring_distal, origin xyz=0.0009359 0 0.028002 rpy=0 0 0, axis 0 1 0, limit lower=0 upper=1.277039 effort=0 velocity=3.1, mimic joint=rh_ring_mcp_pitch multiplier=1.125676 offset=0
- added joint rh_ring_mcp_pitch: type revolute, parent rh_hand_base_link, child rh_ring_proximal, origin xyz=-0.00067368 -0.006217 0.11872 rpy=0.017453 0 0, axis 0 1 0, limit lower=0 upper=1.134464 effort=0.574 velocity=6.10
- added joint rh_ring_tip_fixed: type fixed, parent rh_ring_distal, child rh_ring_tip, origin xyz=0.0341 0 0.034 rpy=0 0 0
- added joint rh_thumb_cmc_pitch: type revolute, parent rh_thumb_metacarpals_base1, child rh_thumb_metacarpals, origin xyz=0.0054997 0.013314 0.0032166 rpy=-1.0762 0.013637 -0.40121, axis 1 0 0, limit lower=0 upper=0.837758 effort=1.008 velocity=3.47
- added joint rh_thumb_cmc_roll: type revolute, parent rh_hand_base_link, child rh_thumb_metacarpals_base1, origin xyz=0.0078133 0.030812 0.025678 rpy=-0.034907 0 0, axis 0 0.034899 -0.99939, limit lower=-0.087266 upper=1.256637 effort=0.588 velocity=5.95
- added joint rh_thumb_dip: type revolute, parent rh_thumb_metacarpals, child rh_thumb_distal, origin xyz=0 -0.0061 0.0827 rpy=0 0 0, axis 1 0 0, limit lower=0 upper=0.963287 effort=0 velocity=1.7, mimic joint=rh_thumb_cmc_pitch multiplier=1.226495 offset=0
- added joint rh_thumb_tip_fixed: type fixed, parent rh_thumb_distal, child rh_thumb_tip, origin xyz=0 -0.0035 0.026 rpy=0 0 -1.5708
