Commit message: Tune PD gains and added OSC control

File: assets/urdf/AR5_L6_description/archive/AR5_L6_workstation.urdf (robot description, URDF)
Before this commit: robot AR5_L6_workstation, 54 links, 53 joints
Joints:
- joint workstation_to_left_arm_base: origin xyz=0.0637 0.715 1.267 rpy=-1.5708 1.5708 0 -> xyz=0.0637 0.716 1.267 rpy=-1.5708 1.5708 0

Commit message: Updated URDF to include camera mount

File: assets/urdf/AR5_L6_description/archive/AR5_L6_workstation.urdf (robot description, URDF)
Before this commit: robot AR5_L6_workstation, 54 links, 53 joints
Links:
- added link camera, mass 0.170230158191785; collision mesh filename=../../camera.STL; visual mesh filename=../../camera.STL
- added link camera_base_link, mass 0.120253078965696; collision mesh filename=../../camera_base_link.STL; visual mesh filename=../../camera_base_link.STL
Joints:
- added joint cameraBase: type fixed, parent workstation_link, child camera_base_link, origin xyz=0.0335 0.67 1.2974 rpy=-1.5708 0 -1.5708, axis 0 0 0
- added joint cameraJoint: type fixed, parent camera_base_link, child camera, origin xyz=0.0801999999999972 0.193139853702623 -0.275851476149329 rpy=-1.26599037580869 -0.643554017997773 -1.5707963267949, axis 0 0 0

File: assets/urdf/workstation.urdf (robot description, URDF)
Before this commit: robot workstation, 1 links, 0 joints
Links:
- added link camera, mass 0.170230158191785; collision mesh filename=camera.STL; visual mesh filename=camera.STL
- added link camera_base_link, mass 0.120253078965696; collision mesh filename=camera_base_link.STL; visual mesh filename=camera_base_link.STL
Joints:
- added joint cameraBase: type fixed, parent workstation_link, child camera_base_link, origin xyz=0.0335 0.67 1.2974 rpy=-1.5708 0 -1.5708, axis 0 0 0
- added joint cameraJoint: type fixed, parent camera_base_link, child camera, origin xyz=0.0801999999999972 0.193139853702623 -0.275851476149329 rpy=-1.26599037580869 -0.643554017997773 -1.5707963267949, axis 0 0 0
