Commit message: Bugfix: Updated workstation URDF recipe and orientation

File: assets/workstations/ar5_l6_bench_bimanual/workstation.urdf (robot description, URDF)
Before this commit: robot ar5_l6_bench_bimanual, 58 links, 57 joints
Joints:
- joint mount_hand_right_to_arm_right_wrist_mount: origin xyz=0 0 0.03 rpy=0 0 1.5708 -> xyz=0 0 0.03 rpy=0 0 -1.5708

File: assets/workstations/ar5_l6_bench_right/workstation.urdf (robot description, URDF)
Before this commit: robot ar5_l6_bench_right, 32 links, 31 joints
Joints:
- joint mount_hand_to_arm_wrist_mount: origin xyz=0 0 0.03 rpy=0 0 1.5708 -> xyz=0 0 0.03 rpy=0 0 -1.5708
