Commit message: fix(a7_lite): use truth URDF joint axes/limits/origins for replay parity
Replay was getting joint-clamped because L1/L2/L4 and R1/R2/R4 had flipped axes and negated/swapped limits relative to the per-side URDF the recorder uses. Also fixed L3/R3 and L4/R4 origin Z (12 mm off). Inertials, masses, and torso mount pads kept (different base STL).

File: assets/components/arms/a7_lite/variants/left/arm.urdf (robot description, URDF)
Before this commit: robot a7_lite_left, 8 links, 7 joints
Joints:
- joint L1_Joint: axis 0 1 0 -> 0 -1 0; limit lower=-3.752 upper=2.181 effort=80 velocity=10.47 -> lower=-2.18 upper=3.75 effort=60 velocity=18.84
- joint L2_Joint: axis 1 0 0 -> -1 0 0; limit lower=-0.148 upper=2.967 effort=80 velocity=10.47 -> lower=-3.33 upper=0.19 effort=60 velocity=18.84
- joint L3_Joint: limit lower=-2.268 upper=2.268 effort=80 velocity=10.47 -> lower=-2.26 upper=2.26 effort=17 velocity=137.68; origin xyz=-0.03125 0 -0.15924 rpy=0 0 0 -> xyz=-0.03125 0 -0.147 rpy=0 0 0
- joint L4_Joint: axis 0 1 0 -> 0 -1 0; limit lower=-1.701 upper=0.785 effort=36 velocity=9.1 -> lower=-0.78 upper=1.74 effort=36 velocity=10.47; origin xyz=0 0.027 -0.11376 rpy=0 0 0 -> xyz=0 0.027 -0.126 rpy=0 0 0
- joint L5_Joint: limit lower=-2.967 upper=2.967 effort=36 velocity=9.1 -> lower=-2.96 upper=2.96 effort=14 velocity=27.21
- joint L6_Joint: limit lower=-1.57 upper=1.57 effort=18 velocity=7.33 -> lower=-1.57 upper=1.57 effort=14 velocity=27.21
- joint L7_Joint: limit lower=-1.57 upper=1.57 effort=18 velocity=7.33 -> lower=-1.57 upper=1.57 effort=14 velocity=27.21; origin xyz=0.0282 -0.028 -0.075 rpy=0 0 0 -> xyz=0.028 -0.028 -0.075 rpy=0 0 0

File: assets/components/arms/a7_lite/variants/right/arm.urdf (robot description, URDF)
Before this commit: robot a7_lite_right, 8 links, 7 joints
Joints:
- joint R1_Joint: axis 0 -1 0 -> 0 1 0; limit lower=-2.181 upper=3.752 effort=80 velocity=10.47 -> lower=-3.75 upper=2.18 effort=60 velocity=18.84
- joint R2_Joint: axis 1 0 0 -> -1 0 0; limit lower=-2.967 upper=0.148 effort=80 velocity=10.47 -> lower=-0.19 upper=3.33 effort=60 velocity=18.84
- joint R3_Joint: limit lower=-2.268 upper=2.268 effort=80 velocity=10.47 -> lower=-2.26 upper=2.26 effort=17 velocity=37.68; origin xyz=-0.03125 0 -0.15924 rpy=0 0 0 -> xyz=-0.03125 0 -0.147 rpy=0 0 0
- joint R4_Joint: axis 0 -1 0 -> 0 1 0; limit lower=-0.785 upper=1.701 effort=36 velocity=9.1 -> lower=-1.74 upper=0.78 effort=36 velocity=10.47; origin xyz=0 -0.027 -0.11376 rpy=0 0 0 -> xyz=0 -0.027 -0.126 rpy=0 0 0
- joint R5_Joint: limit lower=-2.967 upper=2.967 effort=36 velocity=9.1 -> lower=-2.96 upper=2.96 effort=14 velocity=27.21
- joint R6_Joint: limit lower=-1.57 upper=1.57 effort=18 velocity=7.33 -> lower=-1.57 upper=1.57 effort=14 velocity=27.21
- joint R7_Joint: limit lower=-1.57 upper=1.57 effort=18 velocity=7.33 -> lower=-1.57 upper=1.57 effort=14 velocity=27.21; origin xyz=0.0282 0.028 -0.075 rpy=0 0 0 -> xyz=0.028 0.028 -0.075 rpy=0 0 0

File: assets/workstations/a7_lite_dc/workstation.urdf (robot description, URDF)
Before this commit: robot a7_lite_dc, 55 links, 54 joints
Joints:
- joint arm_left_L1_Joint: axis 0 1 0 -> 0 -1 0; limit lower=-3.752 upper=2.181 effort=80 velocity=10.47 -> lower=-2.18 upper=3.75 effort=60 velocity=18.84
- joint arm_left_L2_Joint: axis 1 0 0 -> -1 0 0; limit lower=-0.148 upper=2.967 effort=80 velocity=10.47 -> lower=-3.33 upper=0.19 effort=60 velocity=18.84
- joint arm_left_L3_Joint: limit lower=-2.268 upper=2.268 effort=80 velocity=10.47 -> lower=-2.26 upper=2.26 effort=17 velocity=137.68; origin xyz=-0.03125 0 -0.15924 rpy=0 0 0 -> xyz=-0.03125 0 -0.147 rpy=0 0 0
- joint arm_left_L4_Joint: axis 0 1 0 -> 0 -1 0; limit lower=-1.701 upper=0.785 effort=36 velocity=9.1 -> lower=-0.78 upper=1.74 effort=36 velocity=10.47; origin xyz=0 0.027 -0.11376 rpy=0 0 0 -> xyz=0 0.027 -0.126 rpy=0 0 0
- joint arm_left_L5_Joint: limit lower=-2.967 upper=2.967 effort=36 velocity=9.1 -> lower=-2.96 upper=2.96 effort=14 velocity=27.21
- joint arm_left_L6_Joint: limit lower=-1.57 upper=1.57 effort=18 velocity=7.33 -> lower=-1.57 upper=1.57 effort=14 velocity=27.21
- joint arm_left_L7_Joint: limit lower=-1.57 upper=1.57 effort=18 velocity=7.33 -> lower=-1.57 upper=1.57 effort=14 velocity=27.21; origin xyz=0.0282 -0.028 -0.075 rpy=0 0 0 -> xyz=0.028 -0.028 -0.075 rpy=0 0 0
- joint arm_right_R1_Joint: axis 0 -1 0 -> 0 1 0; limit lower=-2.181 upper=3.752 effort=80 velocity=10.47 -> lower=-3.75 upper=2.18 effort=60 velocity=18.84
- joint arm_right_R2_Joint: axis 1 0 0 -> -1 0 0; limit lower=-2.967 upper=0.148 effort=80 velocity=10.47 -> lower=-0.19 upper=3.33 effort=60 velocity=18.84
- joint arm_right_R3_Joint: limit lower=-2.268 upper=2.268 effort=80 velocity=10.47 -> lower=-2.26 upper=2.26 effort=17 velocity=37.68; origin xyz=-0.03125 0 -0.15924 rpy=0 0 0 -> xyz=-0.03125 0 -0.147 rpy=0 0 0
- joint arm_right_R4_Joint: axis 0 -1 0 -> 0 1 0; limit lower=-0.785 upper=1.701 effort=36 velocity=9.1 -> lower=-1.74 upper=0.78 effort=36 velocity=10.47; origin xyz=0 -0.027 -0.11376 rpy=0 0 0 -> xyz=0 -0.027 -0.126 rpy=0 0 0
- joint arm_right_R5_Joint: limit lower=-2.967 upper=2.967 effort=36 velocity=9.1 -> lower=-2.96 upper=2.96 effort=14 velocity=27.21
- joint arm_right_R6_Joint: limit lower=-1.57 upper=1.57 effort=18 velocity=7.33 -> lower=-1.57 upper=1.57 effort=14 velocity=27.21
- joint arm_right_R7_Joint: limit lower=-1.57 upper=1.57 effort=18 velocity=7.33 -> lower=-1.57 upper=1.57 effort=14 velocity=27.21; origin xyz=0.0282 0.028 -0.075 rpy=0 0 0 -> xyz=0.028 0.028 -0.075 rpy=0 0 0
