Commit message: chore(osc): stub out untested OSC controller, switch default to joint_pd

File: assets/workstations/a7_lite_dc/workstation.urdf (robot description, URDF)
Before this commit: robot a7_lite_dc, 55 links, 54 joints
Joints:
- joint mount_hand_left_to_arm_left_wrist_mount: origin xyz=0 0 0 rpy=3.1416 0 -1.5708 -> xyz=-0.028 0 -0.052 rpy=3.1416 0 -1.5708
- joint mount_hand_right_to_arm_right_wrist_mount: origin xyz=0 0 0 rpy=3.1416 0 1.5708 -> xyz=-0.028 0 -0.052 rpy=3.1416 0 1.5708

File: assets/workstations/a7_lite_o6_dc/workstation.urdf (robot description, URDF)
Before this commit: robot a7_lite_o6_dc, 45 links, 44 joints
Joints:
- joint mount_hand_left_to_arm_left_wrist_mount: origin xyz=0 0 0 rpy=3.1416 0 -1.5708 -> xyz=-0.028 0 -0.052 rpy=3.1416 0 -1.5708
- joint mount_hand_right_to_arm_right_wrist_mount: origin xyz=0 0 0 rpy=3.1416 0 1.5708 -> xyz=-0.028 0 -0.052 rpy=3.1416 0 1.5708
