Commit message: fix(lkls73_arm): normalize all joint axes to match a7_lite convention
Flip axes on all mismatched joints (J1–J7) so lkls73 uses the same sign convention as a7_lite (validated with real-robot replay). Also moves MuJoCo damping from actuator kv (explicit, unstable) to joint damping (implicit, stable).

File: assets/components/arms/lkls73_arm/variants/left/arm.urdf (robot description, URDF)
Before this commit: robot lkls73_arm_left, 9 links, 8 joints
Joints:
- joint L1_Joint: axis 0 1 0 -> 0 -1 0
- joint L2_Joint: axis 1 0 0 -> -1 0 0; limit lower=-0.07 upper=3.2 effort=80 velocity=10.47 -> lower=-3.2 upper=0.07 effort=80 velocity=10.47
- joint L3_Joint: axis 0 0 -1 -> 0 0 1
- joint L4_Joint: axis 0 1 0 -> 0 -1 0
- joint L5_Joint: axis 0 0 -1 -> 0 0 1
- joint L6_Joint: axis 0 1 0 -> 0 -1 0
- joint L7_Joint: axis 1 0 0 -> -1 0 0

File: assets/components/arms/lkls73_arm/variants/right/arm.urdf (robot description, URDF)
Before this commit: robot lkls73_arm_right, 9 links, 8 joints
Joints:
- joint R1_Joint: axis 0 -1 0 -> 0 1 0
- joint R2_Joint: axis 1 0 0 -> -1 0 0; limit lower=-3.2 upper=0.07 effort=80 velocity=10.47 -> lower=-0.07 upper=3.2 effort=80 velocity=10.47
- joint R3_Joint: axis 0 0 -1 -> 0 0 1
- joint R5_Joint: axis 0 0 -1 -> 0 0 1
- joint R7_Joint: axis 1 0 0 -> -1 0 0

File: assets/workstations/lkls73_i1_bimanual/workstation.urdf (robot description, URDF)
Before this commit: robot lkls73_i1_bimanual, 57 links, 56 joints
Joints:
- joint arm_left_L1_Joint: axis 0 1 0 -> 0 -1 0
- joint arm_left_L2_Joint: axis 1 0 0 -> -1 0 0; limit lower=-0.07 upper=3.2 effort=80 velocity=10.47 -> lower=-3.2 upper=0.07 effort=80 velocity=10.47
- joint arm_left_L3_Joint: axis 0 0 -1 -> 0 0 1
- joint arm_left_L4_Joint: axis 0 1 0 -> 0 -1 0
- joint arm_left_L5_Joint: axis 0 0 -1 -> 0 0 1
- joint arm_left_L6_Joint: axis 0 1 0 -> 0 -1 0
- joint arm_left_L7_Joint: axis 1 0 0 -> -1 0 0
- joint arm_right_R1_Joint: axis 0 -1 0 -> 0 1 0
- joint arm_right_R2_Joint: axis 1 0 0 -> -1 0 0; limit lower=-3.2 upper=0.07 effort=80 velocity=10.47 -> lower=-0.07 upper=3.2 effort=80 velocity=10.47
- joint arm_right_R3_Joint: axis 0 0 -1 -> 0 0 1
- joint arm_right_R5_Joint: axis 0 0 -1 -> 0 0 1
- joint arm_right_R7_Joint: axis 1 0 0 -> -1 0 0

File: assets/workstations/lkls73_i1_o6_bimanual/workstation.urdf (robot description, URDF)
Before this commit: robot lkls73_i1_o6_bimanual, 47 links, 46 joints
Joints:
- joint arm_left_L1_Joint: axis 0 1 0 -> 0 -1 0
- joint arm_left_L2_Joint: axis 1 0 0 -> -1 0 0; limit lower=-0.07 upper=3.2 effort=80 velocity=10.47 -> lower=-3.2 upper=0.07 effort=80 velocity=10.47
- joint arm_left_L3_Joint: axis 0 0 -1 -> 0 0 1
- joint arm_left_L4_Joint: axis 0 1 0 -> 0 -1 0
- joint arm_left_L5_Joint: axis 0 0 -1 -> 0 0 1
- joint arm_left_L6_Joint: axis 0 1 0 -> 0 -1 0
- joint arm_left_L7_Joint: axis 1 0 0 -> -1 0 0
- joint arm_right_R1_Joint: axis 0 -1 0 -> 0 1 0
- joint arm_right_R2_Joint: axis 1 0 0 -> -1 0 0; limit lower=-3.2 upper=0.07 effort=80 velocity=10.47 -> lower=-0.07 upper=3.2 effort=80 velocity=10.47
- joint arm_right_R3_Joint: axis 0 0 -1 -> 0 0 1
- joint arm_right_R5_Joint: axis 0 0 -1 -> 0 0 1
- joint arm_right_R7_Joint: axis 1 0 0 -> -1 0 0
