Commit message: fix(assets/ar5_08): align arm parametrization with vendor horizon-install URDF
The in-repo URDF/MJCF had removed the world→base rpy=±π/2 and tried to
compensate via flipped joint axes/origins. The reparametrization shifted
joint_2 zero by ~90° (vendor [-2.0944, 2.0944] vs in-repo [-0.5236, 3.6652]),
so real-robot replay logs rendered ~90° off. Inertials were also swapped
for borrowed 07-class values under a false "vendor ships no inertials" claim.

Port left/right arm.urdf and arm.mjcf to vendor axes, origins, limits,
J4 velocity, and vendor 08-class inertials. tcp z-offset flipped to +0.09.
Joint/link names kept (underscored) for composer compatibility. Recomposed
ar5_08_o6_bench_bimanual and ar5_08_l25_bench_bimanual workstations.

File: packages/linker-robot-assets/src/linker_robot_assets/assets/components/arms/ar5_08/variants/left/arm.urdf (robot description, URDF)
Before this commit: robot arm, 9 links, 8 joints
Links:
- link AR5_5_08L_W4C4A6_link1: mass 2.683 -> 2.166
- link AR5_5_08L_W4C4A6_link2: mass 2.3 -> 1.903
- link AR5_5_08L_W4C4A6_link3: mass 1.862 -> 1.845
- link AR5_5_08L_W4C4A6_link4: mass 1.234 -> 1.037
- link AR5_5_08L_W4C4A6_link5: mass 1.329 -> 1.279
- link AR5_5_08L_W4C4A6_link6: mass 0.93 -> 0.906
Joints:
- joint AR5_5_08L_W4C4A6_joint_1: axis 0 1 0 -> 0 0 1; origin xyz=0.0 0.0 0.0 rpy=0 0 0 -> xyz=0.0 0.0 0.0 rpy=-1.5708 0 0
- joint AR5_5_08L_W4C4A6_joint_2: axis 1 0 0 -> 0 1 0; limit lower=-0.5236 upper=3.6652 effort=108 velocity=3.0543261909900763 -> lower=-2.0944 upper=2.0944 effort=108 velocity=3.0543261909900763; origin xyz=0.0 0.1745 0.0 rpy=0 0 0 -> xyz=0.0 0.0 0.1745 rpy=0 0 0
- joint AR5_5_08L_W4C4A6_joint_3: axis 0 0 -1 -> 0 0 1; origin xyz=0.0 0.0 -0.332 rpy=0 0 0 -> xyz=0.0 0.0 0.332 rpy=0 0 0
- joint AR5_5_08L_W4C4A6_joint_4: axis 0 -1 0 -> 0 1 0; limit lower=-1.0472 upper=2.5307 effort=66 velocity=4.71238898038469 -> lower=-1.0472 upper=2.5307 effort=66 velocity=5.235987755982989
- joint AR5_5_08L_W4C4A6_joint_5: axis 0 0 -1 -> 0 0 1; origin xyz=-0.0105 0.0 -0.278 rpy=0 0 0 -> xyz=-0.0105 0.0 0.278 rpy=0 0 0
- joint AR5_5_08L_W4C4A6_joint_6: axis 0 -1 0 -> 0 1 0
- joint AR5_5_08L_W4C4A6_tcp_joint: origin xyz=0.0 0.0 -0.09 rpy=0 0 0 -> xyz=0.0 0.0 0.09 rpy=0 0 0

File: packages/linker-robot-assets/src/linker_robot_assets/assets/components/arms/ar5_08/variants/right/arm.urdf (robot description, URDF)
Before this commit: robot arm, 9 links, 8 joints
Links:
- link AR5_5_08R_W4C4A6_link1: mass 2.683 -> 2.166
- link AR5_5_08R_W4C4A6_link2: mass 2.3 -> 1.903
- link AR5_5_08R_W4C4A6_link3: mass 1.862 -> 1.845
- link AR5_5_08R_W4C4A6_link4: mass 1.234 -> 1.037
- link AR5_5_08R_W4C4A6_link5: mass 1.329 -> 1.279
- link AR5_5_08R_W4C4A6_link6: mass 0.93 -> 0.906
Joints:
- joint AR5_5_08R_W4C4A6_joint_1: axis 0 -1 0 -> 0 0 1; origin xyz=0.0 0.0 0.0 rpy=0 0 0 -> xyz=0.0 0.0 0.0 rpy=1.5708 0 0
- joint AR5_5_08R_W4C4A6_joint_2: axis 1 0 0 -> 0 1 0; limit lower=-3.6652 upper=0.5236 effort=108 velocity=3.0543261909900763 -> lower=-2.0944 upper=2.0944 effort=108 velocity=3.0543261909900763; origin xyz=0.0 -0.1745 0.0 rpy=0 0 0 -> xyz=0.0 0.0 0.1745 rpy=0 0 0
- joint AR5_5_08R_W4C4A6_joint_3: axis 0 0 -1 -> 0 0 1; origin xyz=0.0 0.0 -0.332 rpy=0 0 0 -> xyz=0.0 0.0 0.332 rpy=0 0 0
- joint AR5_5_08R_W4C4A6_joint_4: axis 0 -1 0 -> 0 1 0; limit lower=-1.0472 upper=2.5307 effort=66 velocity=4.71238898038469 -> lower=-1.0472 upper=2.5307 effort=66 velocity=5.235987755982989
- joint AR5_5_08R_W4C4A6_joint_5: axis 0 0 -1 -> 0 0 1; origin xyz=-0.0105 0.0 -0.278 rpy=0 0 0 -> xyz=-0.0105 0.0 0.278 rpy=0 0 0
- joint AR5_5_08R_W4C4A6_joint_6: axis 0 -1 0 -> 0 1 0
- joint AR5_5_08R_W4C4A6_tcp_joint: origin xyz=0.0 0.0 -0.09 rpy=0 0 0 -> xyz=0.0 0.0 0.09 rpy=0 0 0

File: packages/linker-robot-assets/src/linker_robot_assets/assets/workstations/ar5_08_l25_bench_bimanual/workstation.urdf (robot description, URDF)
Before this commit: robot ar5_08_l25_bench_bimanual, 68 links, 67 joints
Links:
- link arm_left_AR5_5_08L_W4C4A6_link1: mass 2.683 -> 2.166
- link arm_left_AR5_5_08L_W4C4A6_link2: mass 2.3 -> 1.903
- link arm_left_AR5_5_08L_W4C4A6_link3: mass 1.862 -> 1.845
- link arm_left_AR5_5_08L_W4C4A6_link4: mass 1.234 -> 1.037
- link arm_left_AR5_5_08L_W4C4A6_link5: mass 1.329 -> 1.279
- link arm_left_AR5_5_08L_W4C4A6_link6: mass 0.93 -> 0.906
- link arm_right_AR5_5_08R_W4C4A6_link1: mass 2.683 -> 2.166
- link arm_right_AR5_5_08R_W4C4A6_link2: mass 2.3 -> 1.903
- link arm_right_AR5_5_08R_W4C4A6_link3: mass 1.862 -> 1.845
- link arm_right_AR5_5_08R_W4C4A6_link4: mass 1.234 -> 1.037
- link arm_right_AR5_5_08R_W4C4A6_link5: mass 1.329 -> 1.279
- link arm_right_AR5_5_08R_W4C4A6_link6: mass 0.93 -> 0.906
Joints:
- joint arm_left_AR5_5_08L_W4C4A6_joint_1: axis 0 1 0 -> 0 0 1; origin xyz=0 0 0 rpy=0 0 0 -> xyz=0 0 0 rpy=-1.5708 0 0
- joint arm_left_AR5_5_08L_W4C4A6_joint_2: axis 1 0 0 -> 0 1 0; limit lower=-0.5236 upper=3.6652 effort=108 velocity=3.0543261909900763 -> lower=-2.0944 upper=2.0944 effort=108 velocity=3.0543261909900763; origin xyz=0 0.1745 0 rpy=0 0 0 -> xyz=0 0 0.1745 rpy=0 0 0
- joint arm_left_AR5_5_08L_W4C4A6_joint_3: axis 0 0 -1 -> 0 0 1; origin xyz=0 0 -0.332 rpy=0 0 0 -> xyz=0 0 0.332 rpy=0 0 0
- joint arm_left_AR5_5_08L_W4C4A6_joint_4: axis 0 -1 0 -> 0 1 0; limit lower=-1.0472 upper=2.5307 effort=66 velocity=4.71238898038469 -> lower=-1.0472 upper=2.5307 effort=66 velocity=5.235987755982989
- joint arm_left_AR5_5_08L_W4C4A6_joint_5: axis 0 0 -1 -> 0 0 1; origin xyz=-0.0105 0 -0.278 rpy=0 0 0 -> xyz=-0.0105 0 0.278 rpy=0 0 0
- joint arm_left_AR5_5_08L_W4C4A6_joint_6: axis 0 -1 0 -> 0 1 0
- joint arm_left_AR5_5_08L_W4C4A6_tcp_joint: origin xyz=0 0 -0.09 rpy=0 0 0 -> xyz=0 0 0.09 rpy=0 0 0
- joint arm_right_AR5_5_08R_W4C4A6_joint_1: axis 0 -1 0 -> 0 0 1; origin xyz=0 0 0 rpy=0 0 0 -> xyz=0 0 0 rpy=1.5708 0 0
- joint arm_right_AR5_5_08R_W4C4A6_joint_2: axis 1 0 0 -> 0 1 0; limit lower=-3.6652 upper=0.5236 effort=108 velocity=3.0543261909900763 -> lower=-2.0944 upper=2.0944 effort=108 velocity=3.0543261909900763; origin xyz=0 -0.1745 0 rpy=0 0 0 -> xyz=0 0 0.1745 rpy=0 0 0
- joint arm_right_AR5_5_08R_W4C4A6_joint_3: axis 0 0 -1 -> 0 0 1; origin xyz=0 0 -0.332 rpy=0 0 0 -> xyz=0 0 0.332 rpy=0 0 0
- joint arm_right_AR5_5_08R_W4C4A6_joint_4: axis 0 -1 0 -> 0 1 0; limit lower=-1.0472 upper=2.5307 effort=66 velocity=4.71238898038469 -> lower=-1.0472 upper=2.5307 effort=66 velocity=5.235987755982989
- joint arm_right_AR5_5_08R_W4C4A6_joint_5: axis 0 0 -1 -> 0 0 1; origin xyz=-0.0105 0 -0.278 rpy=0 0 0 -> xyz=-0.0105 0 0.278 rpy=0 0 0
- joint arm_right_AR5_5_08R_W4C4A6_joint_6: axis 0 -1 0 -> 0 1 0
- joint arm_right_AR5_5_08R_W4C4A6_tcp_joint: origin xyz=0 0 -0.09 rpy=0 0 0 -> xyz=0 0 0.09 rpy=0 0 0

File: packages/linker-robot-assets/src/linker_robot_assets/assets/workstations/ar5_08_o6_bench_bimanual/workstation.urdf (robot description, URDF)
Before this commit: robot ar5_08_o6_bench_bimanual, 48 links, 47 joints
Links:
- link arm_left_AR5_5_08L_W4C4A6_link1: mass 2.683 -> 2.166
- link arm_left_AR5_5_08L_W4C4A6_link2: mass 2.3 -> 1.903
- link arm_left_AR5_5_08L_W4C4A6_link3: mass 1.862 -> 1.845
- link arm_left_AR5_5_08L_W4C4A6_link4: mass 1.234 -> 1.037
- link arm_left_AR5_5_08L_W4C4A6_link5: mass 1.329 -> 1.279
- link arm_left_AR5_5_08L_W4C4A6_link6: mass 0.93 -> 0.906
- link arm_right_AR5_5_08R_W4C4A6_link1: mass 2.683 -> 2.166
- link arm_right_AR5_5_08R_W4C4A6_link2: mass 2.3 -> 1.903
- link arm_right_AR5_5_08R_W4C4A6_link3: mass 1.862 -> 1.845
- link arm_right_AR5_5_08R_W4C4A6_link4: mass 1.234 -> 1.037
- link arm_right_AR5_5_08R_W4C4A6_link5: mass 1.329 -> 1.279
- link arm_right_AR5_5_08R_W4C4A6_link6: mass 0.93 -> 0.906
Joints:
- joint arm_left_AR5_5_08L_W4C4A6_joint_1: axis 0 1 0 -> 0 0 1; origin xyz=0 0 0 rpy=0 0 0 -> xyz=0 0 0 rpy=-1.5708 0 0
- joint arm_left_AR5_5_08L_W4C4A6_joint_2: axis 1 0 0 -> 0 1 0; limit lower=-0.5236 upper=3.6652 effort=108 velocity=3.0543261909900763 -> lower=-2.0944 upper=2.0944 effort=108 velocity=3.0543261909900763; origin xyz=0 0.1745 0 rpy=0 0 0 -> xyz=0 0 0.1745 rpy=0 0 0
- joint arm_left_AR5_5_08L_W4C4A6_joint_3: axis 0 0 -1 -> 0 0 1; origin xyz=0 0 -0.332 rpy=0 0 0 -> xyz=0 0 0.332 rpy=0 0 0
- joint arm_left_AR5_5_08L_W4C4A6_joint_4: axis 0 -1 0 -> 0 1 0; limit lower=-1.0472 upper=2.5307 effort=66 velocity=4.71238898038469 -> lower=-1.0472 upper=2.5307 effort=66 velocity=5.235987755982989
- joint arm_left_AR5_5_08L_W4C4A6_joint_5: axis 0 0 -1 -> 0 0 1; origin xyz=-0.0105 0 -0.278 rpy=0 0 0 -> xyz=-0.0105 0 0.278 rpy=0 0 0
- joint arm_left_AR5_5_08L_W4C4A6_joint_6: axis 0 -1 0 -> 0 1 0
- joint arm_left_AR5_5_08L_W4C4A6_tcp_joint: origin xyz=0 0 -0.09 rpy=0 0 0 -> xyz=0 0 0.09 rpy=0 0 0
- joint arm_right_AR5_5_08R_W4C4A6_joint_1: axis 0 -1 0 -> 0 0 1; origin xyz=0 0 0 rpy=0 0 0 -> xyz=0 0 0 rpy=1.5708 0 0
- joint arm_right_AR5_5_08R_W4C4A6_joint_2: axis 1 0 0 -> 0 1 0; limit lower=-3.6652 upper=0.5236 effort=108 velocity=3.0543261909900763 -> lower=-2.0944 upper=2.0944 effort=108 velocity=3.0543261909900763; origin xyz=0 -0.1745 0 rpy=0 0 0 -> xyz=0 0 0.1745 rpy=0 0 0
- joint arm_right_AR5_5_08R_W4C4A6_joint_3: axis 0 0 -1 -> 0 0 1; origin xyz=0 0 -0.332 rpy=0 0 0 -> xyz=0 0 0.332 rpy=0 0 0
- joint arm_right_AR5_5_08R_W4C4A6_joint_4: axis 0 -1 0 -> 0 1 0; limit lower=-1.0472 upper=2.5307 effort=66 velocity=4.71238898038469 -> lower=-1.0472 upper=2.5307 effort=66 velocity=5.235987755982989
- joint arm_right_AR5_5_08R_W4C4A6_joint_5: axis 0 0 -1 -> 0 0 1; origin xyz=-0.0105 0 -0.278 rpy=0 0 0 -> xyz=-0.0105 0 0.278 rpy=0 0 0
- joint arm_right_AR5_5_08R_W4C4A6_joint_6: axis 0 -1 0 -> 0 1 0
- joint arm_right_AR5_5_08R_W4C4A6_tcp_joint: origin xyz=0 0 -0.09 rpy=0 0 0 -> xyz=0 0 0.09 rpy=0 0 0
