Commit message: feat(assets/linkerhand_o6): swap to GLB visuals + voxel-hull OBJ collision; flatten layout; fix left thumb
- URDFs: visual=.glb, collision=voxel-hull .obj (~190 KB/side vs ~10 MB STL)
- Left thumb joints rebuilt from new SolidWorks export (cmc_yaw axis 0,0,1→0,1,0;
  cmc_pitch + ip pos/euler/axis updated; mimic 2.29→1.8788) — fixes prior 180° error
- hand.mjcf → hand.xml; per-link visual .obj from Blender's direct GLB export
- Flatten variants/<side>/ tree: URDFs/XMLs at component root, shared meshes/
  with {lh,rh}_*_{vis,col}.{glb,obj} prefix-suffix naming so every file is
  globally unique (online viewers no longer conflate left/right same-named meshes)
- All 4 O6 workstations re-composed; component + workstation + drift gates green

File: packages/linker-robot-assets/src/linker_robot_assets/assets/workstations/a7_lite_o6_dc/workstation.urdf (robot description, URDF)
Before this commit: robot a7_lite_o6_dc, 45 links, 44 joints
Links:
- link hand_left_lh_hand_base_link: geometry collision mesh filename=../../components/hands/linkerhand_o6/meshes/collision/lh_ha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; visual mesh filename=../../components/hands/linkerhand_o6/meshes/visual/lh_hand_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
- link hand_left_lh_index_distal: geometry collision mesh filename=../../components/hands/linkerhand_o6/meshes/collision/lh_in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; visual mesh filename=../../components/hands/linkerhand_o6/meshes/visual/lh_index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
- link hand_left_lh_index_proximal: geometry collision mesh filename=../../components/hands/linkerhand_o6/meshes/collision/lh_in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; visual mesh filename=../../components/hands/linkerhand_o6/meshes/visual/lh_index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
- link hand_left_lh_middle_distal: geometry collision mesh filename=../../components/hands/linkerhand_o6/meshes/collision/lh_mi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; visual mesh filename=../../components/hands/linkerhand_o6/meshes/visual/lh_middl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
- link hand_left_lh_middle_proximal: geometry collision mesh filename=../../components/hands/linkerhand_o6/meshes/collision/lh_mi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; visual mesh filename=../../components/hands/linkerhand_o6/meshes/visual/lh_middl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
- link hand_left_lh_pinky_distal: geometry collision mesh filename=../../components/hands/linkerhand_o6/meshes/collision/lh_pi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; visual mesh filename=../../components/hands/linkerhand_o6/meshes/visual/lh_pinky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
- link hand_left_lh_pinky_proximal: geometry collision mesh filename=../../components/hands/linkerhand_o6/meshes/collision/lh_pi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; visual mesh filename=../../components/hands/linkerhand_o6/meshes/visual/lh_pinky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
- link hand_left_lh_ring_distal: geometry collision mesh filename=../../components/hands/linkerhand_o6/meshes/collision/lh_ri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; visual mesh filename=../../components/hands/linkerhand_o6/meshes/visual/lh_ring_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
- link hand_left_lh_ring_proximal: geometry collision mesh filename=../../components/hands/linkerhand_o6/meshes/collision/lh_ri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; visual mesh filename=../../components/hands/linkerhand_o6/meshes/visual/lh_ring_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
- link hand_left_lh_thumb_distal: geometry collision mesh filename=../../components/hands/linkerhand_o6/meshes/collision/lh_th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; visual mesh filename=../../components/hands/linkerhand_o6/meshes/visual/lh_thumb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
- link hand_left_lh_thumb_metacarpals: geometry collision mesh filename=../../components/hands/linkerhand_o6/meshes/collision/lh_th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; visual mesh filename=../../components/hands/linkerhand_o6/meshes/visual/lh_thumb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
- link hand_left_lh_thumb_metacarpals_base2: geometry collision mesh filename=../../components/hands/linkerhand_o6/meshes/collision/lh_th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; visual mesh filename=../../components/hands/linkerhand_o6/meshes/visual/lh_thumb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
- link hand_right_rh_hand_base_link: geometry collision mesh filename=../../components/hands/linkerhand_o6/meshes/collision/rh_ha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; visual mesh filename=../../components/hands/linkerhand_o6/meshes/visual/rh_hand_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
- link hand_right_rh_index_distal: geometry collision mesh filename=../../components/hands/linkerhand_o6/meshes/collision/rh_in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; visual mesh filename=../../components/hands/linkerhand_o6/meshes/visual/rh_index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
- link hand_right_rh_index_proximal: geometry collision mesh filename=../../components/hands/linkerhand_o6/meshes/collision/rh_in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; visual mesh filename=../../components/hands/linkerhand_o6/meshes/visual/rh_index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
- link hand_right_rh_middle_distal: geometry collision mesh filename=../../components/hands/linkerhand_o6/meshes/collision/rh_mi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; visual mesh filename=../../components/hands/linkerhand_o6/meshes/visual/rh_middl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
- link hand_right_rh_middle_proximal: geometry collision mesh filename=../../components/hands/linkerhand_o6/meshes/collision/rh_mi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; visual mesh filename=../../components/hands/linkerhand_o6/meshes/visual/rh_middl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
- link hand_right_rh_pinky_distal: geometry collision mesh filename=../../components/hands/linkerhand_o6/meshes/collision/rh_pi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; visual mesh filename=../../components/hands/linkerhand_o6/meshes/visual/rh_pinky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
- link hand_right_rh_pinky_proximal: geometry collision mesh filename=../../components/hands/linkerhand_o6/meshes/collision/rh_pi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; visual mesh filename=../../components/hands/linkerhand_o6/meshes/visual/rh_pinky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
- link hand_right_rh_ring_distal: geometry collision mesh filename=../../components/hands/linkerhand_o6/meshes/collision/rh_ri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; visual mesh filename=../../components/hands/linkerhand_o6/meshes/visual/rh_ring_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
- link hand_right_rh_ring_proximal: geometry collision mesh filename=../../components/hands/linkerhand_o6/meshes/collision/rh_ri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; visual mesh filename=../../components/hands/linkerhand_o6/meshes/visual/rh_ring_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
- link hand_right_rh_thumb_distal: geometry collision mesh filename=../../components/hands/linkerhand_o6/meshes/collision/rh_th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; visual mesh filename=../../components/hands/linkerhand_o6/meshes/visual/rh_thumb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
- link hand_right_rh_thumb_metacarpals: geometry collision mesh filename=../../components/hands/linkerhand_o6/meshes/collision/rh_th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; visual mesh filename=../../components/hands/linkerhand_o6/meshes/visual/rh_thumb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
- link hand_right_rh_thumb_metacarpals_base2: geometry collision mesh filename=../../components/hands/linkerhand_o6/meshes/collision/rh_th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; visual mesh filename=../../components/hands/linkerhand_o6/meshes/visual/rh_thumb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
Joints:
- joint hand_left_lh_thumb_cmc_pitch: axis 0 1 0 -> 0 -1 0; origin xyz=0.0061649 -0.010678 -0.004891 rpy=0 -1.1529 2.0944 -> xyz=0.00915604684 -0.00603785696 0.0158587383 rpy=-0.575786024 -0.407073695 -1.31922273
- joint hand_left_lh_thumb_cmc_yaw: axis 0 0 1 -> 0 1 0; origin xyz=0.011508 -0.022975 0.032794 rpy=0 0 0 -> xyz=0.0115084536 -0.022975 0.030794 rpy=1.57079633 0 0
- joint hand_left_lh_thumb_ip: axis 0 1 0 -> 0 -1 0; mimic joint=hand_left_lh_thumb_cmc_pitch multiplier=2.29 offset=0 -> joint=hand_left_lh_thumb_cmc_pitch multiplier=1.8788 offset=0; origin xyz=0.0037776 0 0.045368 rpy=0 0 0 -> xyz=0 0 0.036812 rpy=0 0 0

File: packages/linker-robot-assets/src/linker_robot_assets/assets/workstations/ar5_08_o6_bench_bimanual/workstation.urdf (robot description, URDF)
Before this commit: robot ar5_08_o6_bench_bimanual, 48 links, 47 joints
Links:
- link hand_left_lh_hand_base_link: geometry collision mesh filename=../../components/hands/linkerhand_o6/meshes/collision/lh_ha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; visual mesh filename=../../components/hands/linkerhand_o6/meshes/visual/lh_hand_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
- link hand_left_lh_index_distal: geometry collision mesh filename=../../components/hands/linkerhand_o6/meshes/collision/lh_in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; visual mesh filename=../../components/hands/linkerhand_o6/meshes/visual/lh_index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
- link hand_left_lh_index_proximal: geometry collision mesh filename=../../components/hands/linkerhand_o6/meshes/collision/lh_in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; visual mesh filename=../../components/hands/linkerhand_o6/meshes/visual/lh_index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
- link hand_left_lh_middle_distal: geometry collision mesh filename=../../components/hands/linkerhand_o6/meshes/collision/lh_mi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; visual mesh filename=../../components/hands/linkerhand_o6/meshes/visual/lh_middl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
- link hand_left_lh_middle_proximal: geometry collision mesh filename=../../components/hands/linkerhand_o6/meshes/collision/lh_mi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; visual mesh filename=../../components/hands/linkerhand_o6/meshes/visual/lh_middl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
- link hand_left_lh_pinky_distal: geometry collision mesh filename=../../components/hands/linkerhand_o6/meshes/collision/lh_pi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; visual mesh filename=../../components/hands/linkerhand_o6/meshes/visual/lh_pinky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
- link hand_left_lh_pinky_proximal: geometry collision mesh filename=../../components/hands/linkerhand_o6/meshes/collision/lh_pi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; visual mesh filename=../../components/hands/linkerhand_o6/meshes/visual/lh_pinky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
- link hand_left_lh_ring_distal: geometry collision mesh filename=../../components/hands/linkerhand_o6/meshes/collision/lh_ri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; visual mesh filename=../../components/hands/linkerhand_o6/meshes/visual/lh_ring_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
- link hand_left_lh_ring_proximal: geometry collision mesh filename=../../components/hands/linkerhand_o6/meshes/collision/lh_ri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; visual mesh filename=../../components/hands/linkerhand_o6/meshes/visual/lh_ring_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
- link hand_left_lh_thumb_distal: geometry collision mesh filename=../../components/hands/linkerhand_o6/meshes/collision/lh_th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; visual mesh filename=../../components/hands/linkerhand_o6/meshes/visual/lh_thumb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
- link hand_left_lh_thumb_metacarpals: geometry collision mesh filename=../../components/hands/linkerhand_o6/meshes/collision/lh_th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; visual mesh filename=../../components/hands/linkerhand_o6/meshes/visual/lh_thumb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
- link hand_left_lh_thumb_metacarpals_base2: geometry collision mesh filename=../../components/hands/linkerhand_o6/meshes/collision/lh_th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; visual mesh filename=../../components/hands/linkerhand_o6/meshes/visual/lh_thumb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
- link hand_right_rh_hand_base_link: geometry collision mesh filename=../../components/hands/linkerhand_o6/meshes/collision/rh_ha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; visual mesh filename=../../components/hands/linkerhand_o6/meshes/visual/rh_hand_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
- link hand_right_rh_index_distal: geometry collision mesh filename=../../components/hands/linkerhand_o6/meshes/collision/rh_in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; visual mesh filename=../../components/hands/linkerhand_o6/meshes/visual/rh_index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
- link hand_right_rh_index_proximal: geometry collision mesh filename=../../components/hands/linkerhand_o6/meshes/collision/rh_in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; visual mesh filename=../../components/hands/linkerhand_o6/meshes/visual/rh_index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
- link hand_right_rh_middle_distal: geometry collision mesh filename=../../components/hands/linkerhand_o6/meshes/collision/rh_mi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; visual mesh filename=../../components/hands/linkerhand_o6/meshes/visual/rh_middl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
- link hand_right_rh_middle_proximal: geometry collision mesh filename=../../components/hands/linkerhand_o6/meshes/collision/rh_mi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; visual mesh filename=../../components/hands/linkerhand_o6/meshes/visual/rh_middl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
- link hand_right_rh_pinky_distal: geometry collision mesh filename=../../components/hands/linkerhand_o6/meshes/collision/rh_pi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; visual mesh filename=../../components/hands/linkerhand_o6/meshes/visual/rh_pinky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
- link hand_right_rh_pinky_proximal: geometry collision mesh filename=../../components/hands/linkerhand_o6/meshes/collision/rh_pi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; visual mesh filename=../../components/hands/linkerhand_o6/meshes/visual/rh_pinky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
- link hand_right_rh_ring_distal: geometry collision mesh filename=../../components/hands/linkerhand_o6/meshes/collision/rh_ri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; visual mesh filename=../../components/hands/linkerhand_o6/meshes/visual/rh_ring_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
- link hand_right_rh_ring_proximal: geometry collision mesh filename=../../components/hands/linkerhand_o6/meshes/collision/rh_ri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; visual mesh filename=../../components/hands/linkerhand_o6/meshes/visual/rh_ring_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
- link hand_right_rh_thumb_distal: geometry collision mesh filename=../../components/hands/linkerhand_o6/meshes/collision/rh_th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; visual mesh filename=../../components/hands/linkerhand_o6/meshes/visual/rh_thumb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
- link hand_right_rh_thumb_metacarpals: geometry collision mesh filename=../../components/hands/linkerhand_o6/meshes/collision/rh_th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; visual mesh filename=../../components/hands/linkerhand_o6/meshes/visual/rh_thumb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
- link hand_right_rh_thumb_metacarpals_base2: geometry collision mesh filename=../../components/hands/linkerhand_o6/meshes/collision/rh_th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; visual mesh filename=../../components/hands/linkerhand_o6/meshes/visual/rh_thumb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
Joints:
- joint hand_left_lh_thumb_cmc_pitch: axis 0 1 0 -> 0 -1 0; origin xyz=0.0061649 -0.010678 -0.004891 rpy=0 -1.1529 2.0944 -> xyz=0.00915604684 -0.00603785696 0.0158587383 rpy=-0.575786024 -0.407073695 -1.31922273
- joint hand_left_lh_thumb_cmc_yaw: axis 0 0 1 -> 0 1 0; origin xyz=0.011508 -0.022975 0.032794 rpy=0 0 0 -> xyz=0.0115084536 -0.022975 0.030794 rpy=1.57079633 0 0
- joint hand_left_lh_thumb_ip: axis 0 1 0 -> 0 -1 0; mimic joint=hand_left_lh_thumb_cmc_pitch multiplier=2.29 offset=0 -> joint=hand_left_lh_thumb_cmc_pitch multiplier=1.8788 offset=0; origin xyz=0.0037776 0 0.045368 rpy=0 0 0 -> xyz=0 0 0.036812 rpy=0 0 0

File: packages/linker-robot-assets/src/linker_robot_assets/assets/workstations/ar5_o6_bench_bimanual/workstation.urdf (robot description, URDF)
Before this commit: robot ar5_o6_bench_bimanual, 48 links, 47 joints
Links:
- link hand_left_lh_hand_base_link: geometry collision mesh filename=../../components/hands/linkerhand_o6/meshes/collision/lh_ha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; visual mesh filename=../../components/hands/linkerhand_o6/meshes/visual/lh_hand_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
- link hand_left_lh_index_distal: geometry collision mesh filename=../../components/hands/linkerhand_o6/meshes/collision/lh_in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; visual mesh filename=../../components/hands/linkerhand_o6/meshes/visual/lh_index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
- link hand_left_lh_index_proximal: geometry collision mesh filename=../../components/hands/linkerhand_o6/meshes/collision/lh_in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; visual mesh filename=../../components/hands/linkerhand_o6/meshes/visual/lh_index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
- link hand_left_lh_middle_distal: geometry collision mesh filename=../../components/hands/linkerhand_o6/meshes/collision/lh_mi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; visual mesh filename=../../components/hands/linkerhand_o6/meshes/visual/lh_middl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
- link hand_left_lh_middle_proximal: geometry collision mesh filename=../../components/hands/linkerhand_o6/meshes/collision/lh_mi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; visual mesh filename=../../components/hands/linkerhand_o6/meshes/visual/lh_middl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
- link hand_left_lh_pinky_distal: geometry collision mesh filename=../../components/hands/linkerhand_o6/meshes/collision/lh_pi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; visual mesh filename=../../components/hands/linkerhand_o6/meshes/visual/lh_pinky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
- link hand_left_lh_pinky_proximal: geometry collision mesh filename=../../components/hands/linkerhand_o6/meshes/collision/lh_pi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; visual mesh filename=../../components/hands/linkerhand_o6/meshes/visual/lh_pinky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
- link hand_left_lh_ring_distal: geometry collision mesh filename=../../components/hands/linkerhand_o6/meshes/collision/lh_ri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; visual mesh filename=../../components/hands/linkerhand_o6/meshes/visual/lh_ring_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
- link hand_left_lh_ring_proximal: geometry collision mesh filename=../../components/hands/linkerhand_o6/meshes/collision/lh_ri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; visual mesh filename=../../components/hands/linkerhand_o6/meshes/visual/lh_ring_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
- link hand_left_lh_thumb_distal: geometry collision mesh filename=../../components/hands/linkerhand_o6/meshes/collision/lh_th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; visual mesh filename=../../components/hands/linkerhand_o6/meshes/visual/lh_thumb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
- link hand_left_lh_thumb_metacarpals: geometry collision mesh filename=../../components/hands/linkerhand_o6/meshes/collision/lh_th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; visual mesh filename=../../components/hands/linkerhand_o6/meshes/visual/lh_thumb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
- link hand_left_lh_thumb_metacarpals_base2: geometry collision mesh filename=../../components/hands/linkerhand_o6/meshes/collision/lh_th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; visual mesh filename=../../components/hands/linkerhand_o6/meshes/visual/lh_thumb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
- link hand_right_rh_hand_base_link: geometry collision mesh filename=../../components/hands/linkerhand_o6/meshes/collision/rh_ha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; visual mesh filename=../../components/hands/linkerhand_o6/meshes/visual/rh_hand_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
- link hand_right_rh_index_distal: geometry collision mesh filename=../../components/hands/linkerhand_o6/meshes/collision/rh_in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; visual mesh filename=../../components/hands/linkerhand_o6/meshes/visual/rh_index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
- link hand_right_rh_index_proximal: geometry collision mesh filename=../../components/hands/linkerhand_o6/meshes/collision/rh_in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; visual mesh filename=../../components/hands/linkerhand_o6/meshes/visual/rh_index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
- link hand_right_rh_middle_distal: geometry collision mesh filename=../../components/hands/linkerhand_o6/meshes/collision/rh_mi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; visual mesh filename=../../components/hands/linkerhand_o6/meshes/visual/rh_middl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
- link hand_right_rh_middle_proximal: geometry collision mesh filename=../../components/hands/linkerhand_o6/meshes/collision/rh_mi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; visual mesh filename=../../components/hands/linkerhand_o6/meshes/visual/rh_middl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
- link hand_right_rh_pinky_distal: geometry collision mesh filename=../../components/hands/linkerhand_o6/meshes/collision/rh_pi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; visual mesh filename=../../components/hands/linkerhand_o6/meshes/visual/rh_pinky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
- link hand_right_rh_pinky_proximal: geometry collision mesh filename=../../components/hands/linkerhand_o6/meshes/collision/rh_pi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; visual mesh filename=../../components/hands/linkerhand_o6/meshes/visual/rh_pinky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
- link hand_right_rh_ring_distal: geometry collision mesh filename=../../components/hands/linkerhand_o6/meshes/collision/rh_ri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; visual mesh filename=../../components/hands/linkerhand_o6/meshes/visual/rh_ring_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
- link hand_right_rh_ring_proximal: geometry collision mesh filename=../../components/hands/linkerhand_o6/meshes/collision/rh_ri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; visual mesh filename=../../components/hands/linkerhand_o6/meshes/visual/rh_ring_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
- link hand_right_rh_thumb_distal: geometry collision mesh filename=../../components/hands/linkerhand_o6/meshes/collision/rh_th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; visual mesh filename=../../components/hands/linkerhand_o6/meshes/visual/rh_thumb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
- link hand_right_rh_thumb_metacarpals: geometry collision mesh filename=../../components/hands/linkerhand_o6/meshes/collision/rh_th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; visual mesh filename=../../components/hands/linkerhand_o6/meshes/visual/rh_thumb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
- link hand_right_rh_thumb_metacarpals_base2: geometry collision mesh filename=../../components/hands/linkerhand_o6/meshes/collision/rh_th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; visual mesh filename=../../components/hands/linkerhand_o6/meshes/visual/rh_thumb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
Joints:
- joint hand_left_lh_thumb_cmc_pitch: axis 0 1 0 -> 0 -1 0; origin xyz=0.0061649 -0.010678 -0.004891 rpy=0 -1.1529 2.0944 -> xyz=0.00915604684 -0.00603785696 0.0158587383 rpy=-0.575786024 -0.407073695 -1.31922273
- joint hand_left_lh_thumb_cmc_yaw: axis 0 0 1 -> 0 1 0; origin xyz=0.011508 -0.022975 0.032794 rpy=0 0 0 -> xyz=0.0115084536 -0.022975 0.030794 rpy=1.57079633 0 0
- joint hand_left_lh_thumb_ip: axis 0 1 0 -> 0 -1 0; mimic joint=hand_left_lh_thumb_cmc_pitch multiplier=2.29 offset=0 -> joint=hand_left_lh_thumb_cmc_pitch multiplier=1.8788 offset=0; origin xyz=0.0037776 0 0.045368 rpy=0 0 0 -> xyz=0 0 0.036812 rpy=0 0 0
