Commit message: feat(assets): add L20Lite hand, refresh L25 URDF, add a7_lite_l20lite_dc
- New linkerhand_l20lite component (10 actuated + 10 mimic per variant)
- L25 refreshed from 2026-06-25 vendor drop: thumb_ip→thumb_dip, retuned
  mimic multipliers and joint limits, flipped finger mcp_roll axes;
  auto-patched thumb_metacarpals_base2 inertia to satisfy MuJoCo's
  triangle inequality
- Recomposed all 4 L25-consuming workstations
- Added a7_lite_l20lite_dc workstation + Hydra robot config

File: packages/linker-robot-assets/src/linker_robot_assets/assets/workstations/ar5_l25_bench_bimanual/workstation.urdf (robot description, URDF)
Before this commit: robot ar5_l25_bench_bimanual, 68 links, 67 joints
Joints:
- removed joint hand_left_lh_thumb_ip
- removed joint hand_right_rh_thumb_ip
- added joint hand_left_lh_thumb_dip: type revolute, parent hand_left_lh_thumb_proximal, child hand_left_lh_thumb_distal, origin xyz=-0.00483652209 0 0.0342226492 rpy=0 0 0, axis 0 1 0, limit lower=0 upper=1.2392 effort=100 velocity=1, mimic joint=hand_left_lh_thumb_mcp multiplier=1.0142 offset=0
- added joint hand_right_rh_thumb_dip: type revolute, parent hand_right_rh_thumb_proximal, child hand_right_rh_thumb_distal, origin xyz=-0.0048365 0 0.034223 rpy=0 0 0, axis 0 1 0, limit lower=0 upper=1.2392 effort=1 velocity=100, mimic joint=hand_right_rh_thumb_mcp multiplier=1.0142 offset=0
- joint hand_left_lh_index_dip: limit lower=0 upper=1.55 effort=100 velocity=1 -> lower=0 upper=1.3614 effort=100 velocity=1; mimic joint=hand_left_lh_index_pip multiplier=0.89 offset=0 -> joint=hand_left_lh_index_pip multiplier=0.7879 offset=0
- joint hand_left_lh_index_mcp_pitch: limit lower=0 upper=1.22 effort=100 velocity=1 -> lower=0 upper=1.2217 effort=100 velocity=1
- joint hand_left_lh_index_mcp_roll: axis 1 0 0 -> -1 0 0; limit lower=-0.23 upper=0.23 effort=100 velocity=1 -> lower=-0.2269 upper=0.2269 effort=100 velocity=1
- joint hand_left_lh_index_pip: limit lower=0 upper=1.74 effort=100 velocity=1 -> lower=0 upper=1.7279 effort=100 velocity=1
- joint hand_left_lh_middle_dip: limit lower=0 upper=1.55 effort=100 velocity=1 -> lower=0 upper=1.3614 effort=100 velocity=1; mimic joint=hand_left_lh_middle_pip multiplier=0.89 offset=0 -> joint=hand_left_lh_middle_pip multiplier=0.7879 offset=0
- joint hand_left_lh_middle_mcp_pitch: limit lower=0 upper=1.22 effort=100 velocity=1 -> lower=0 upper=1.2217 effort=100 velocity=1
- joint hand_left_lh_middle_mcp_roll: axis 1 0 0 -> -1 0 0
- joint hand_left_lh_middle_pip: limit lower=0 upper=1.74 effort=100 velocity=1 -> lower=0 upper=1.7279 effort=100 velocity=1
- joint hand_left_lh_pinky_dip: limit lower=0 upper=1.55 effort=100 velocity=1 -> lower=0 upper=1.3614 effort=100 velocity=1; mimic joint=hand_left_lh_pinky_pip multiplier=0.89 offset=0 -> joint=hand_left_lh_pinky_pip multiplier=0.7879 offset=0
- joint hand_left_lh_pinky_mcp_pitch: limit lower=0 upper=1.22 effort=100 velocity=1 -> lower=0 upper=1.2217 effort=100 velocity=1
- joint hand_left_lh_pinky_mcp_roll: axis 1 0 0 -> -1 0 0
- joint hand_left_lh_pinky_pip: limit lower=0 upper=1.74 effort=100 velocity=1 -> lower=0 upper=1.7279 effort=100 velocity=1
- joint hand_left_lh_ring_dip: limit lower=0 upper=1.55 effort=100 velocity=1 -> lower=0 upper=1.3614 effort=100 velocity=1; mimic joint=hand_left_lh_ring_pip multiplier=0.89 offset=0 -> joint=hand_left_lh_ring_pip multiplier=0.7879 offset=0
- joint hand_left_lh_ring_mcp_pitch: limit lower=0 upper=1.22 effort=100 velocity=1 -> lower=0 upper=1.2217 effort=100 velocity=1
- joint hand_left_lh_ring_mcp_roll: axis 1 0 0 -> -1 0 0
- joint hand_left_lh_ring_pip: limit lower=0 upper=1.74 effort=100 velocity=1 -> lower=0 upper=1.7279 effort=100 velocity=1
- joint hand_left_lh_thumb_cmc_pitch: limit lower=0 upper=0.84 effort=100 velocity=1 -> lower=0 upper=0.7854 effort=100 velocity=1; origin xyz=0.0088218 -0.024245 0.0005 rpy=0 -1.0647 1.9199 -> xyz=0.0088218 -0.024245 0.0005 rpy=0 -0.91 1.9199
- joint hand_left_lh_thumb_cmc_roll: limit lower=0 upper=1.4 effort=100 velocity=1 -> lower=0 upper=1.309 effort=100 velocity=1
- joint hand_left_lh_thumb_cmc_yaw: limit lower=0 upper=1.57 effort=100 velocity=1 -> lower=0 upper=1.5882 effort=100 velocity=1
- joint hand_left_lh_thumb_mcp: limit lower=0 upper=1.26 effort=100 velocity=1 -> lower=0 upper=1.2217 effort=100 velocity=1
- joint hand_right_rh_index_dip: limit lower=0 upper=1.55 effort=1 velocity=100 -> lower=0 upper=1.3614 effort=1 velocity=100; mimic joint=hand_right_rh_index_pip multiplier=0.89 offset=0 -> joint=hand_right_rh_index_pip multiplier=0.7879 offset=0
- joint hand_right_rh_index_mcp_pitch: limit lower=0 upper=1.22 effort=1 velocity=100 -> lower=0 upper=1.2217 effort=1 velocity=100
- joint hand_right_rh_index_mcp_roll: axis 1 0 0 -> -1 0 0; limit lower=-0.23 upper=0.23 effort=1 velocity=100 -> lower=-0.2269 upper=0.2269 effort=1 velocity=100
- joint hand_right_rh_index_pip: limit lower=0 upper=1.75 effort=1 velocity=100 -> lower=0 upper=1.7279 effort=1 velocity=100
- joint hand_right_rh_middle_dip: limit lower=0 upper=1.55 effort=1 velocity=100 -> lower=0 upper=1.3614 effort=1 velocity=100; mimic joint=hand_right_rh_middle_pip multiplier=0.89 offset=0 -> joint=hand_right_rh_middle_pip multiplier=0.7879 offset=0
- joint hand_right_rh_middle_mcp_pitch: limit lower=0 upper=1.22 effort=1 velocity=100 -> lower=0 upper=1.2217 effort=1 velocity=100
- joint hand_right_rh_middle_mcp_roll: axis 1 0 0 -> -1 0 0
- joint hand_right_rh_middle_pip: limit lower=0 upper=1.75 effort=1 velocity=100 -> lower=0 upper=1.7279 effort=1 velocity=100
- joint hand_right_rh_pinky_dip: limit lower=0 upper=1.55 effort=1 velocity=100 -> lower=0 upper=1.3614 effort=1 velocity=100; mimic joint=hand_right_rh_pinky_pip multiplier=0.89 offset=0 -> joint=hand_right_rh_pinky_pip multiplier=0.7879 offset=0
- joint hand_right_rh_pinky_mcp_pitch: limit lower=0 upper=1.22 effort=1 velocity=100 -> lower=0 upper=1.2217 effort=1 velocity=100
- joint hand_right_rh_pinky_mcp_roll: axis 1 0 0 -> -1 0 0
- joint hand_right_rh_pinky_pip: limit lower=0 upper=1.75 effort=1 velocity=100 -> lower=0 upper=1.7279 effort=1 velocity=100
- joint hand_right_rh_ring_dip: limit lower=0 upper=1.55 effort=1 velocity=100 -> lower=0 upper=1.3614 effort=1 velocity=100; mimic joint=hand_right_rh_ring_pip multiplier=0.89 offset=0 -> joint=hand_right_rh_ring_pip multiplier=0.7879 offset=0
- joint hand_right_rh_ring_mcp_pitch: limit lower=0 upper=1.22 effort=1 velocity=100 -> lower=0 upper=1.2217 effort=1 velocity=100
- joint hand_right_rh_ring_mcp_roll: axis 1 0 0 -> -1 0 0
- joint hand_right_rh_ring_pip: limit lower=0 upper=1.75 effort=1 velocity=100 -> lower=0 upper=1.7279 effort=1 velocity=100
- joint hand_right_rh_thumb_cmc_pitch: limit lower=0 upper=0.83 effort=1 velocity=100 -> lower=0 upper=0.7854 effort=1 velocity=100; origin xyz=0.0088264 0.024243 0.0005 rpy=0 -1.0647 -1.9199 -> xyz=0.0088264 0.024243 0.0005 rpy=0 -0.91 -1.9199
- joint hand_right_rh_thumb_cmc_roll: limit lower=0 upper=1.39 effort=1 velocity=100 -> lower=0 upper=1.309 effort=1 velocity=100
- joint hand_right_rh_thumb_cmc_yaw: limit lower=0 upper=1.57 effort=1 velocity=100 -> lower=0 upper=1.5882 effort=1 velocity=100
- joint hand_right_rh_thumb_mcp: limit lower=0 upper=1.25 effort=1 velocity=100 -> lower=0 upper=1.2217 effort=1 velocity=100

File: packages/linker-robot-assets/src/linker_robot_assets/assets/workstations/lkls73_i1_l25_bimanual/workstation.urdf (robot description, URDF)
Before this commit: robot lkls73_i1_l25_bimanual, 67 links, 66 joints
Joints:
- removed joint hand_left_lh_thumb_ip
- removed joint hand_right_rh_thumb_ip
- added joint hand_left_lh_thumb_dip: type revolute, parent hand_left_lh_thumb_proximal, child hand_left_lh_thumb_distal, origin xyz=-0.00483652209 0 0.0342226492 rpy=0 0 0, axis 0 1 0, limit lower=0 upper=1.2392 effort=100 velocity=1, mimic joint=hand_left_lh_thumb_mcp multiplier=1.0142 offset=0
- added joint hand_right_rh_thumb_dip: type revolute, parent hand_right_rh_thumb_proximal, child hand_right_rh_thumb_distal, origin xyz=-0.0048365 0 0.034223 rpy=0 0 0, axis 0 1 0, limit lower=0 upper=1.2392 effort=1 velocity=100, mimic joint=hand_right_rh_thumb_mcp multiplier=1.0142 offset=0
- joint hand_left_lh_index_dip: limit lower=0 upper=1.55 effort=100 velocity=1 -> lower=0 upper=1.3614 effort=100 velocity=1; mimic joint=hand_left_lh_index_pip multiplier=0.89 offset=0 -> joint=hand_left_lh_index_pip multiplier=0.7879 offset=0
- joint hand_left_lh_index_mcp_pitch: limit lower=0 upper=1.22 effort=100 velocity=1 -> lower=0 upper=1.2217 effort=100 velocity=1
- joint hand_left_lh_index_mcp_roll: axis 1 0 0 -> -1 0 0; limit lower=-0.23 upper=0.23 effort=100 velocity=1 -> lower=-0.2269 upper=0.2269 effort=100 velocity=1
- joint hand_left_lh_index_pip: limit lower=0 upper=1.74 effort=100 velocity=1 -> lower=0 upper=1.7279 effort=100 velocity=1
- joint hand_left_lh_middle_dip: limit lower=0 upper=1.55 effort=100 velocity=1 -> lower=0 upper=1.3614 effort=100 velocity=1; mimic joint=hand_left_lh_middle_pip multiplier=0.89 offset=0 -> joint=hand_left_lh_middle_pip multiplier=0.7879 offset=0
- joint hand_left_lh_middle_mcp_pitch: limit lower=0 upper=1.22 effort=100 velocity=1 -> lower=0 upper=1.2217 effort=100 velocity=1
- joint hand_left_lh_middle_mcp_roll: axis 1 0 0 -> -1 0 0
- joint hand_left_lh_middle_pip: limit lower=0 upper=1.74 effort=100 velocity=1 -> lower=0 upper=1.7279 effort=100 velocity=1
- joint hand_left_lh_pinky_dip: limit lower=0 upper=1.55 effort=100 velocity=1 -> lower=0 upper=1.3614 effort=100 velocity=1; mimic joint=hand_left_lh_pinky_pip multiplier=0.89 offset=0 -> joint=hand_left_lh_pinky_pip multiplier=0.7879 offset=0
- joint hand_left_lh_pinky_mcp_pitch: limit lower=0 upper=1.22 effort=100 velocity=1 -> lower=0 upper=1.2217 effort=100 velocity=1
- joint hand_left_lh_pinky_mcp_roll: axis 1 0 0 -> -1 0 0
- joint hand_left_lh_pinky_pip: limit lower=0 upper=1.74 effort=100 velocity=1 -> lower=0 upper=1.7279 effort=100 velocity=1
- joint hand_left_lh_ring_dip: limit lower=0 upper=1.55 effort=100 velocity=1 -> lower=0 upper=1.3614 effort=100 velocity=1; mimic joint=hand_left_lh_ring_pip multiplier=0.89 offset=0 -> joint=hand_left_lh_ring_pip multiplier=0.7879 offset=0
- joint hand_left_lh_ring_mcp_pitch: limit lower=0 upper=1.22 effort=100 velocity=1 -> lower=0 upper=1.2217 effort=100 velocity=1
- joint hand_left_lh_ring_mcp_roll: axis 1 0 0 -> -1 0 0
- joint hand_left_lh_ring_pip: limit lower=0 upper=1.74 effort=100 velocity=1 -> lower=0 upper=1.7279 effort=100 velocity=1
- joint hand_left_lh_thumb_cmc_pitch: limit lower=0 upper=0.84 effort=100 velocity=1 -> lower=0 upper=0.7854 effort=100 velocity=1; origin xyz=0.0088218 -0.024245 0.0005 rpy=0 -1.0647 1.9199 -> xyz=0.0088218 -0.024245 0.0005 rpy=0 -0.91 1.9199
- joint hand_left_lh_thumb_cmc_roll: limit lower=0 upper=1.4 effort=100 velocity=1 -> lower=0 upper=1.309 effort=100 velocity=1
- joint hand_left_lh_thumb_cmc_yaw: limit lower=0 upper=1.57 effort=100 velocity=1 -> lower=0 upper=1.5882 effort=100 velocity=1
- joint hand_left_lh_thumb_mcp: limit lower=0 upper=1.26 effort=100 velocity=1 -> lower=0 upper=1.2217 effort=100 velocity=1
- joint hand_right_rh_index_dip: limit lower=0 upper=1.55 effort=1 velocity=100 -> lower=0 upper=1.3614 effort=1 velocity=100; mimic joint=hand_right_rh_index_pip multiplier=0.89 offset=0 -> joint=hand_right_rh_index_pip multiplier=0.7879 offset=0
- joint hand_right_rh_index_mcp_pitch: limit lower=0 upper=1.22 effort=1 velocity=100 -> lower=0 upper=1.2217 effort=1 velocity=100
- joint hand_right_rh_index_mcp_roll: axis 1 0 0 -> -1 0 0; limit lower=-0.23 upper=0.23 effort=1 velocity=100 -> lower=-0.2269 upper=0.2269 effort=1 velocity=100
- joint hand_right_rh_index_pip: limit lower=0 upper=1.75 effort=1 velocity=100 -> lower=0 upper=1.7279 effort=1 velocity=100
- joint hand_right_rh_middle_dip: limit lower=0 upper=1.55 effort=1 velocity=100 -> lower=0 upper=1.3614 effort=1 velocity=100; mimic joint=hand_right_rh_middle_pip multiplier=0.89 offset=0 -> joint=hand_right_rh_middle_pip multiplier=0.7879 offset=0
- joint hand_right_rh_middle_mcp_pitch: limit lower=0 upper=1.22 effort=1 velocity=100 -> lower=0 upper=1.2217 effort=1 velocity=100
- joint hand_right_rh_middle_mcp_roll: axis 1 0 0 -> -1 0 0
- joint hand_right_rh_middle_pip: limit lower=0 upper=1.75 effort=1 velocity=100 -> lower=0 upper=1.7279 effort=1 velocity=100
- joint hand_right_rh_pinky_dip: limit lower=0 upper=1.55 effort=1 velocity=100 -> lower=0 upper=1.3614 effort=1 velocity=100; mimic joint=hand_right_rh_pinky_pip multiplier=0.89 offset=0 -> joint=hand_right_rh_pinky_pip multiplier=0.7879 offset=0
- joint hand_right_rh_pinky_mcp_pitch: limit lower=0 upper=1.22 effort=1 velocity=100 -> lower=0 upper=1.2217 effort=1 velocity=100
- joint hand_right_rh_pinky_mcp_roll: axis 1 0 0 -> -1 0 0
- joint hand_right_rh_pinky_pip: limit lower=0 upper=1.75 effort=1 velocity=100 -> lower=0 upper=1.7279 effort=1 velocity=100
- joint hand_right_rh_ring_dip: limit lower=0 upper=1.55 effort=1 velocity=100 -> lower=0 upper=1.3614 effort=1 velocity=100; mimic joint=hand_right_rh_ring_pip multiplier=0.89 offset=0 -> joint=hand_right_rh_ring_pip multiplier=0.7879 offset=0
- joint hand_right_rh_ring_mcp_pitch: limit lower=0 upper=1.22 effort=1 velocity=100 -> lower=0 upper=1.2217 effort=1 velocity=100
- joint hand_right_rh_ring_mcp_roll: axis 1 0 0 -> -1 0 0
- joint hand_right_rh_ring_pip: limit lower=0 upper=1.75 effort=1 velocity=100 -> lower=0 upper=1.7279 effort=1 velocity=100
- joint hand_right_rh_thumb_cmc_pitch: limit lower=0 upper=0.83 effort=1 velocity=100 -> lower=0 upper=0.7854 effort=1 velocity=100; origin xyz=0.0088264 0.024243 0.0005 rpy=0 -1.0647 -1.9199 -> xyz=0.0088264 0.024243 0.0005 rpy=0 -0.91 -1.9199
- joint hand_right_rh_thumb_cmc_roll: limit lower=0 upper=1.39 effort=1 velocity=100 -> lower=0 upper=1.309 effort=1 velocity=100
- joint hand_right_rh_thumb_cmc_yaw: limit lower=0 upper=1.57 effort=1 velocity=100 -> lower=0 upper=1.5882 effort=1 velocity=100
- joint hand_right_rh_thumb_mcp: limit lower=0 upper=1.25 effort=1 velocity=100 -> lower=0 upper=1.2217 effort=1 velocity=100
