Commit message: refactor(assets): rename lkls73 → p7 across arm, torso, workstations
Renames the lkls73_arm component to `p7`, lkls73_torso → p7_torso, and the
three lkls73_i1_* workstations to p7_i1_*. Updates all internal identifiers
(URDF robot names, MJCF model + class names, material, recipe/manifest/config
references, docs, and the add_robot_component skill). Recomposes the p7
workstations plus a7_lite dependents so the drift gate is clean.

Refs: #6

File: packages/linker-robot-assets/src/linker_robot_assets/assets/workstations/p7_i1_bimanual/workstation.urdf (robot description, URDF)
Before this commit: robot a7_lite_l6_dc, 55 links, 54 joints
Links:
- added link arm_left_L8_Link, mass 6.05149284897746E-05; collision mesh filename=../../components/arms/p7/variants/left/meshes/L8_Link.STL; visual mesh filename=../../components/arms/p7/variants/left/meshes/L8_Link.STL
- added link arm_right_R8_Link, mass 6.05149284897743E-05; collision mesh filename=../../components/arms/p7/variants/right/meshes/R8_Link.STL; visual mesh filename=../../components/arms/p7/variants/right/meshes/R8_Link.STL
- link arm_left_L1_Link: mass 1.1899 -> 1.3997199601261; geometry collision mesh filename=../../components/arms/p7/variants/left/meshes/L1_Link.STL; visual mesh filename=../../components/arms/p7/variants/left/meshes/L1_Link.STL
- link arm_left_L2_Link: mass 1.0659 -> 1.14210487960353; geometry collision mesh filename=../../components/arms/p7/variants/left/meshes/L2_Link.STL; visual mesh filename=../../components/arms/p7/variants/left/meshes/L2_Link.STL
- link arm_left_L3_Link: mass 1.2763 -> 1.2798435287888; geometry collision mesh filename=../../components/arms/p7/variants/left/meshes/L3_Link.STL; visual mesh filename=../../components/arms/p7/variants/left/meshes/L3_Link.STL
- link arm_left_L4_Link: mass 0.66812 -> 0.935504485205333; geometry collision mesh filename=../../components/arms/p7/variants/left/meshes/L4_Link.STL; visual mesh filename=../../components/arms/p7/variants/left/meshes/L4_Link.STL
- link arm_left_L5_Link: mass 0.4439 -> 0.298012293033296; geometry collision mesh filename=../../components/arms/p7/variants/left/meshes/L5_Link.STL; visual mesh filename=../../components/arms/p7/variants/left/meshes/L5_Link.STL
- link arm_left_L6_Link: mass 0.5193 -> 0.344326210144814; geometry collision mesh filename=../../components/arms/p7/variants/left/meshes/L6_Link.STL; visual mesh filename=../../components/arms/p7/variants/left/meshes/L6_Link.STL
- link arm_left_L7_Link: mass 0.10175 -> 0.143310943627726; geometry collision mesh filename=../../components/arms/p7/variants/left/meshes/L7_Link.STL; visual mesh filename=../../components/arms/p7/variants/left/meshes/L7_Link.STL
- link arm_right_R1_Link: mass 1.1899 -> 1.39972022686362; geometry collision mesh filename=../../components/arms/p7/variants/right/meshes/R1_Link.STL; visual mesh filename=../../components/arms/p7/variants/right/meshes/R1_Link.STL
- link arm_right_R2_Link: mass 1.0663 -> 1.14210467744301; geometry collision mesh filename=../../components/arms/p7/variants/right/meshes/R2_Link.STL; visual mesh filename=../../components/arms/p7/variants/right/meshes/R2_Link.STL
- link arm_right_R3_Link: mass 1.3517 -> 1.27984352653686; geometry collision mesh filename=../../components/arms/p7/variants/right/meshes/R3_Link.STL; visual mesh filename=../../components/arms/p7/variants/right/meshes/R3_Link.STL
- link arm_right_R4_Link: mass 0.69691 -> 0.935504488206621; geometry collision mesh filename=../../components/arms/p7/variants/right/meshes/R4_Link.STL; visual mesh filename=../../components/arms/p7/variants/right/meshes/R4_Link.STL
- link arm_right_R5_Link: mass 0.48527 -> 0.298013716041534; geometry collision mesh filename=../../components/arms/p7/variants/right/meshes/R5_Link.STL; visual mesh filename=../../components/arms/p7/variants/right/meshes/R5_Link.STL
- link arm_right_R6_Link: mass 0.5193 -> 0.344326135276304; geometry collision mesh filename=../../components/arms/p7/variants/right/meshes/R6_Link.STL; visual mesh filename=../../components/arms/p7/variants/right/meshes/R6_Link.STL
- link arm_right_R7_Link: mass 0.10175 -> 0.143310943627727; geometry collision mesh filename=../../components/arms/p7/variants/right/meshes/R7_Link.STL; visual mesh filename=../../components/arms/p7/variants/right/meshes/R7_Link.STL
- link base_base_link: mass 8.6616 -> 10.8067081992573; geometry collision mesh filename=../../components/bases/p7_torso/variants/default/meshes/bas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; visual mesh filename=../../components/bases/p7_torso/variants/default/meshes/bas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
Joints:
- added joint arm_left_L8_Joint: type fixed, parent arm_left_L7_Link, child arm_left_L8_Link, origin xyz=2.5732e-05 0 -0.0455 rpy=0 0 0, axis 0 0 0
- added joint arm_right_R8_Joint: type fixed, parent arm_right_R7_Link, child arm_right_R8_Link, origin xyz=-2.5732e-05 0 -0.0455 rpy=0 0 0, axis 0 0 0
- joint arm_left_L1_Joint: limit lower=-2.18 upper=3.75 effort=60 velocity=18.84 -> lower=-2.91 upper=2.91 effort=80 velocity=10.47
- joint arm_left_L2_Joint: limit lower=-3.33 upper=0.19 effort=60 velocity=18.84 -> lower=-3.2 upper=0.07 effort=80 velocity=10.47; origin xyz=0.03125 0.0715 0 rpy=0 0 0 -> xyz=0 0.058 0 rpy=0 0 0
- joint arm_left_L3_Joint: limit lower=-2.26 upper=2.26 effort=17 velocity=137.68 -> lower=-2.69 upper=2.69 effort=36 velocity=9.1; origin xyz=-0.03125 0 -0.147 rpy=0 0 0 -> xyz=-2.5018e-05 0 -0.123 rpy=0 0 0
- joint arm_left_L4_Joint: limit lower=-0.78 upper=1.74 effort=36 velocity=10.47 -> lower=-2.05 upper=2.05 effort=36 velocity=9.1; origin xyz=0 0.027 -0.126 rpy=0 0 0 -> xyz=2.4267e-05 0 -0.1621 rpy=0 0 0
- joint arm_left_L5_Joint: limit lower=-2.96 upper=2.96 effort=14 velocity=27.21 -> lower=-2.69 upper=2.69 effort=36 velocity=9.1; origin xyz=0 -0.027 -0.136 rpy=0 0 0 -> xyz=0 0 -0.124 rpy=0 0 0
- joint arm_left_L6_Joint: limit lower=-1.57 upper=1.57 effort=14 velocity=27.21 -> lower=-1.59 upper=1.59 effort=18 velocity=7.33; origin xyz=0 0.028 -0.0435 rpy=0 0 0 -> xyz=0 0 -0.0881 rpy=0 0 0
- joint arm_left_L7_Joint: limit lower=-1.57 upper=1.57 effort=14 velocity=27.21 -> lower=-1.59 upper=1.59 effort=18 velocity=7.33; origin xyz=0.028 -0.028 -0.075 rpy=0 0 0 -> xyz=-2.6563e-05 0 -0.0655 rpy=0 0 0
- joint arm_right_R1_Joint: limit lower=-3.75 upper=2.18 effort=60 velocity=18.84 -> lower=-2.91 upper=2.91 effort=80 velocity=10.47
- joint arm_right_R2_Joint: limit lower=-0.19 upper=3.33 effort=60 velocity=18.84 -> lower=-0.07 upper=3.2 effort=80 velocity=10.47; origin xyz=0.03125 -0.0715 0 rpy=0 0 0 -> xyz=-3.32e-05 -0.058001 0 rpy=0 0 0
- joint arm_right_R3_Joint: limit lower=-2.26 upper=2.26 effort=17 velocity=37.68 -> lower=-2.69 upper=2.69 effort=36 velocity=9.1; origin xyz=-0.03125 0 -0.147 rpy=0 0 0 -> xyz=2.5018e-05 0 -0.123 rpy=0 0 0
- joint arm_right_R4_Joint: limit lower=-1.74 upper=0.78 effort=36 velocity=10.47 -> lower=-2.05 upper=2.05 effort=36 velocity=9.1; origin xyz=0 -0.027 -0.126 rpy=0 0 0 -> xyz=-2.5308e-05 0 -0.1621 rpy=0 0 0
- joint arm_right_R5_Joint: limit lower=-2.96 upper=2.96 effort=14 velocity=27.21 -> lower=-2.69 upper=2.69 effort=36 velocity=9.1; origin xyz=0 0.027 -0.136 rpy=0 0 0 -> xyz=0 0 -0.124 rpy=0 0 0
- joint arm_right_R6_Joint: limit lower=-1.57 upper=1.57 effort=14 velocity=27.21 -> lower=-1.59 upper=1.59 effort=18 velocity=7.33; origin xyz=0 -0.028 -0.0435 rpy=0 0 0 -> xyz=0 0 -0.0881 rpy=0 0 0
- joint arm_right_R7_Joint: limit lower=-1.57 upper=1.57 effort=14 velocity=27.21 -> lower=-1.59 upper=1.59 effort=18 velocity=7.33; origin xyz=0.028 0.028 -0.075 rpy=0 0 0 -> xyz=2.5631e-05 0 -0.0655 rpy=0 0 0
- joint base_weld_arm_left_mount: origin xyz=0.0062932 0.1505 -0.022706 rpy=0 0 0 -> xyz=0 0.164 0 rpy=0 0 0
- joint base_weld_arm_right_mount: origin xyz=0.0062926 -0.1505 -0.022706 rpy=0 0 0 -> xyz=3.32e-05 -0.164 0 rpy=0 0 0
- joint mount_hand_left_to_arm_left_wrist_mount: origin xyz=-0.028 0 -0.052 rpy=3.1416 0 -1.5708 -> xyz=0 0 0 rpy=3.1416 0 -1.5708; parent arm_left_L7_Link -> arm_left_L8_Link
- joint mount_hand_right_to_arm_right_wrist_mount: origin xyz=-0.028 0 -0.052 rpy=3.1416 0 1.5708 -> xyz=0 0 0 rpy=3.1416 0 1.5708; parent arm_right_R7_Link -> arm_right_R8_Link

File: packages/linker-robot-assets/src/linker_robot_assets/assets/workstations/p7_i1_o6_bimanual/workstation.urdf (robot description, URDF)
Before this commit: robot a7_lite_o6_dc, 45 links, 44 joints
Links:
- added link arm_left_L8_Link, mass 6.05149284897746E-05; collision mesh filename=../../components/arms/p7/variants/left/meshes/L8_Link.STL; visual mesh filename=../../components/arms/p7/variants/left/meshes/L8_Link.STL
- added link arm_right_R8_Link, mass 6.05149284897743E-05; collision mesh filename=../../components/arms/p7/variants/right/meshes/R8_Link.STL; visual mesh filename=../../components/arms/p7/variants/right/meshes/R8_Link.STL
- link arm_left_L1_Link: mass 1.1899 -> 1.3997199601261; geometry collision mesh filename=../../components/arms/p7/variants/left/meshes/L1_Link.STL; visual mesh filename=../../components/arms/p7/variants/left/meshes/L1_Link.STL
- link arm_left_L2_Link: mass 1.0659 -> 1.14210487960353; geometry collision mesh filename=../../components/arms/p7/variants/left/meshes/L2_Link.STL; visual mesh filename=../../components/arms/p7/variants/left/meshes/L2_Link.STL
- link arm_left_L3_Link: mass 1.2763 -> 1.2798435287888; geometry collision mesh filename=../../components/arms/p7/variants/left/meshes/L3_Link.STL; visual mesh filename=../../components/arms/p7/variants/left/meshes/L3_Link.STL
- link arm_left_L4_Link: mass 0.66812 -> 0.935504485205333; geometry collision mesh filename=../../components/arms/p7/variants/left/meshes/L4_Link.STL; visual mesh filename=../../components/arms/p7/variants/left/meshes/L4_Link.STL
- link arm_left_L5_Link: mass 0.4439 -> 0.298012293033296; geometry collision mesh filename=../../components/arms/p7/variants/left/meshes/L5_Link.STL; visual mesh filename=../../components/arms/p7/variants/left/meshes/L5_Link.STL
- link arm_left_L6_Link: mass 0.5193 -> 0.344326210144814; geometry collision mesh filename=../../components/arms/p7/variants/left/meshes/L6_Link.STL; visual mesh filename=../../components/arms/p7/variants/left/meshes/L6_Link.STL
- link arm_left_L7_Link: mass 0.10175 -> 0.143310943627726; geometry collision mesh filename=../../components/arms/p7/variants/left/meshes/L7_Link.STL; visual mesh filename=../../components/arms/p7/variants/left/meshes/L7_Link.STL
- link arm_right_R1_Link: mass 1.1899 -> 1.39972022686362; geometry collision mesh filename=../../components/arms/p7/variants/right/meshes/R1_Link.STL; visual mesh filename=../../components/arms/p7/variants/right/meshes/R1_Link.STL
- link arm_right_R2_Link: mass 1.0663 -> 1.14210467744301; geometry collision mesh filename=../../components/arms/p7/variants/right/meshes/R2_Link.STL; visual mesh filename=../../components/arms/p7/variants/right/meshes/R2_Link.STL
- link arm_right_R3_Link: mass 1.3517 -> 1.27984352653686; geometry collision mesh filename=../../components/arms/p7/variants/right/meshes/R3_Link.STL; visual mesh filename=../../components/arms/p7/variants/right/meshes/R3_Link.STL
- link arm_right_R4_Link: mass 0.69691 -> 0.935504488206621; geometry collision mesh filename=../../components/arms/p7/variants/right/meshes/R4_Link.STL; visual mesh filename=../../components/arms/p7/variants/right/meshes/R4_Link.STL
- link arm_right_R5_Link: mass 0.48527 -> 0.298013716041534; geometry collision mesh filename=../../components/arms/p7/variants/right/meshes/R5_Link.STL; visual mesh filename=../../components/arms/p7/variants/right/meshes/R5_Link.STL
- link arm_right_R6_Link: mass 0.5193 -> 0.344326135276304; geometry collision mesh filename=../../components/arms/p7/variants/right/meshes/R6_Link.STL; visual mesh filename=../../components/arms/p7/variants/right/meshes/R6_Link.STL
- link arm_right_R7_Link: mass 0.10175 -> 0.143310943627727; geometry collision mesh filename=../../components/arms/p7/variants/right/meshes/R7_Link.STL; visual mesh filename=../../components/arms/p7/variants/right/meshes/R7_Link.STL
- link base_base_link: mass 8.6616 -> 10.8067081992573; geometry collision mesh filename=../../components/bases/p7_torso/variants/default/meshes/bas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; visual mesh filename=../../components/bases/p7_torso/variants/default/meshes/bas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
Joints:
- added joint arm_left_L8_Joint: type fixed, parent arm_left_L7_Link, child arm_left_L8_Link, origin xyz=2.5732e-05 0 -0.0455 rpy=0 0 0, axis 0 0 0
- added joint arm_right_R8_Joint: type fixed, parent arm_right_R7_Link, child arm_right_R8_Link, origin xyz=-2.5732e-05 0 -0.0455 rpy=0 0 0, axis 0 0 0
- joint arm_left_L1_Joint: limit lower=-2.18 upper=3.75 effort=60 velocity=18.84 -> lower=-2.91 upper=2.91 effort=80 velocity=10.47
- joint arm_left_L2_Joint: limit lower=-3.33 upper=0.19 effort=60 velocity=18.84 -> lower=-3.2 upper=0.07 effort=80 velocity=10.47; origin xyz=0.03125 0.0715 0 rpy=0 0 0 -> xyz=0 0.058 0 rpy=0 0 0
- joint arm_left_L3_Joint: limit lower=-2.26 upper=2.26 effort=17 velocity=137.68 -> lower=-2.69 upper=2.69 effort=36 velocity=9.1; origin xyz=-0.03125 0 -0.147 rpy=0 0 0 -> xyz=-2.5018e-05 0 -0.123 rpy=0 0 0
- joint arm_left_L4_Joint: limit lower=-0.78 upper=1.74 effort=36 velocity=10.47 -> lower=-2.05 upper=2.05 effort=36 velocity=9.1; origin xyz=0 0.027 -0.126 rpy=0 0 0 -> xyz=2.4267e-05 0 -0.1621 rpy=0 0 0
- joint arm_left_L5_Joint: limit lower=-2.96 upper=2.96 effort=14 velocity=27.21 -> lower=-2.69 upper=2.69 effort=36 velocity=9.1; origin xyz=0 -0.027 -0.136 rpy=0 0 0 -> xyz=0 0 -0.124 rpy=0 0 0
- joint arm_left_L6_Joint: limit lower=-1.57 upper=1.57 effort=14 velocity=27.21 -> lower=-1.59 upper=1.59 effort=18 velocity=7.33; origin xyz=0 0.028 -0.0435 rpy=0 0 0 -> xyz=0 0 -0.0881 rpy=0 0 0
- joint arm_left_L7_Joint: limit lower=-1.57 upper=1.57 effort=14 velocity=27.21 -> lower=-1.59 upper=1.59 effort=18 velocity=7.33; origin xyz=0.028 -0.028 -0.075 rpy=0 0 0 -> xyz=-2.6563e-05 0 -0.0655 rpy=0 0 0
- joint arm_right_R1_Joint: limit lower=-3.75 upper=2.18 effort=60 velocity=18.84 -> lower=-2.91 upper=2.91 effort=80 velocity=10.47
- joint arm_right_R2_Joint: limit lower=-0.19 upper=3.33 effort=60 velocity=18.84 -> lower=-0.07 upper=3.2 effort=80 velocity=10.47; origin xyz=0.03125 -0.0715 0 rpy=0 0 0 -> xyz=-3.32e-05 -0.058001 0 rpy=0 0 0
- joint arm_right_R3_Joint: limit lower=-2.26 upper=2.26 effort=17 velocity=37.68 -> lower=-2.69 upper=2.69 effort=36 velocity=9.1; origin xyz=-0.03125 0 -0.147 rpy=0 0 0 -> xyz=2.5018e-05 0 -0.123 rpy=0 0 0
- joint arm_right_R4_Joint: limit lower=-1.74 upper=0.78 effort=36 velocity=10.47 -> lower=-2.05 upper=2.05 effort=36 velocity=9.1; origin xyz=0 -0.027 -0.126 rpy=0 0 0 -> xyz=-2.5308e-05 0 -0.1621 rpy=0 0 0
- joint arm_right_R5_Joint: limit lower=-2.96 upper=2.96 effort=14 velocity=27.21 -> lower=-2.69 upper=2.69 effort=36 velocity=9.1; origin xyz=0 0.027 -0.136 rpy=0 0 0 -> xyz=0 0 -0.124 rpy=0 0 0
- joint arm_right_R6_Joint: limit lower=-1.57 upper=1.57 effort=14 velocity=27.21 -> lower=-1.59 upper=1.59 effort=18 velocity=7.33; origin xyz=0 -0.028 -0.0435 rpy=0 0 0 -> xyz=0 0 -0.0881 rpy=0 0 0
- joint arm_right_R7_Joint: limit lower=-1.57 upper=1.57 effort=14 velocity=27.21 -> lower=-1.59 upper=1.59 effort=18 velocity=7.33; origin xyz=0.028 0.028 -0.075 rpy=0 0 0 -> xyz=2.5631e-05 0 -0.0655 rpy=0 0 0
- joint base_weld_arm_left_mount: origin xyz=0.0062932 0.1505 -0.022706 rpy=0 0 0 -> xyz=0 0.164 0 rpy=0 0 0
- joint base_weld_arm_right_mount: origin xyz=0.0062926 -0.1505 -0.022706 rpy=0 0 0 -> xyz=3.32e-05 -0.164 0 rpy=0 0 0
- joint mount_hand_left_to_arm_left_wrist_mount: origin xyz=-0.028 0 -0.052 rpy=3.1416 0 -1.5708 -> xyz=0 0 0 rpy=3.1416 0 -1.5708; parent arm_left_L7_Link -> arm_left_L8_Link
- joint mount_hand_right_to_arm_right_wrist_mount: origin xyz=-0.028 0 -0.052 rpy=3.1416 0 1.5708 -> xyz=0 0 0 rpy=3.1416 0 1.5708; parent arm_right_R7_Link -> arm_right_R8_Link
