Commit message: feat(a7_lite): swap in A7_Lite0812 torso (head+chest) and vendor TCP (#20)
Closes #19

Replace the bare-column base_link with the vendor A7_Lite0812 mesh
(decimated 527k->100k faces for MuJoCo's 200k cap), re-place the stand
so feet rest on the ground and shoulders stay symmetric at +/-0.1505,
and adopt the vendor's exact hand TCP in all four a7_lite_*_dc recipes.
Arms unchanged. Recomposed + validated l6/l25/o6/l20lite.

Reviewed-on: https://gitea.linkerhub.work/LinkerOS/linker-sim/pulls/20
Reviewed-by: 孙煜童 <yutong.sun25@gmail.com>
Co-authored-by: Ryan Zhou <ryanzed12138@gmail.com>
Co-committed-by: Ryan Zhou <ryanzed12138@gmail.com>

File: packages/linker-robot-assets/src/linker_robot_assets/assets/components/bases/a7_lite_torso/variants/default/base.urdf (robot description, URDF)
Before this commit: robot a7_lite_torso, 4 links, 3 joints
Links:
- link base_link: mass 8.6616 -> 11.244; geometry collision mesh filename=meshes/base_link.STL; visual mesh filename=meshes/base_link_visual.STL
Joints:
- joint torso_stand: origin xyz=0 0 1.2 rpy=0 0 0 -> xyz=0 0.01438 1.301489 rpy=0 0 0
- joint weld_arm_left_mount: origin xyz=0.0062932 0.1505 -0.022706 rpy=0 0 0 -> xyz=0 0.13612 0 rpy=0 0 0
- joint weld_arm_right_mount: origin xyz=0.0062926 -0.1505 -0.022706 rpy=0 0 0 -> xyz=0 -0.16488 0 rpy=0 0 0

File: packages/linker-robot-assets/src/linker_robot_assets/assets/workstations/a7_lite_l20lite_dc/workstation.urdf (robot description, URDF)
Before this commit: robot a7_lite_l20lite_dc, 63 links, 62 joints
Links:
- link base_base_link: mass 8.6616 -> 11.244
Joints:
- joint base_torso_stand: origin xyz=0 0 1.2 rpy=0 0 0 -> xyz=0 0.01438 1.301489 rpy=0 0 0
- joint base_weld_arm_left_mount: origin xyz=0.0062932 0.1505 -0.022706 rpy=0 0 0 -> xyz=0 0.13612 0 rpy=0 0 0
- joint base_weld_arm_right_mount: origin xyz=0.0062926 -0.1505 -0.022706 rpy=0 0 0 -> xyz=0 -0.16488 0 rpy=0 0 0
- joint mount_hand_left_to_arm_left_wrist_mount: origin xyz=-0.028 0 -0.052 rpy=3.1416 0 -1.5708 -> xyz=-0.028 0 -0.0525 rpy=3.1416 0 -1.5708
- joint mount_hand_right_to_arm_right_wrist_mount: origin xyz=-0.028 0 -0.052 rpy=3.1416 0 1.5708 -> xyz=-0.0282 0 -0.0527 rpy=3.1416 0 1.5708

File: packages/linker-robot-assets/src/linker_robot_assets/assets/workstations/a7_lite_l25_dc/workstation.urdf (robot description, URDF)
Before this commit: robot a7_lite_l25_dc, 65 links, 64 joints
Links:
- link base_base_link: mass 8.6616 -> 11.244
Joints:
- joint base_torso_stand: origin xyz=0 0 1.2 rpy=0 0 0 -> xyz=0 0.01438 1.301489 rpy=0 0 0
- joint base_weld_arm_left_mount: origin xyz=0.0062932 0.1505 -0.022706 rpy=0 0 0 -> xyz=0 0.13612 0 rpy=0 0 0
- joint base_weld_arm_right_mount: origin xyz=0.0062926 -0.1505 -0.022706 rpy=0 0 0 -> xyz=0 -0.16488 0 rpy=0 0 0
- joint mount_hand_left_to_arm_left_wrist_mount: origin xyz=-0.028 0 -0.052 rpy=3.1416 0 -1.5708 -> xyz=-0.028 0 -0.0525 rpy=3.1416 0 -1.5708
- joint mount_hand_right_to_arm_right_wrist_mount: origin xyz=-0.028 0 -0.052 rpy=3.1416 0 1.5708 -> xyz=-0.0282 0 -0.0527 rpy=3.1416 0 1.5708

File: packages/linker-robot-assets/src/linker_robot_assets/assets/workstations/a7_lite_l6_dc/workstation.urdf (robot description, URDF)
Before this commit: robot a7_lite_l6_dc, 55 links, 54 joints
Links:
- link base_base_link: mass 8.6616 -> 11.244
Joints:
- joint base_torso_stand: origin xyz=0 0 1.2 rpy=0 0 0 -> xyz=0 0.01438 1.301489 rpy=0 0 0
- joint base_weld_arm_left_mount: origin xyz=0.0062932 0.1505 -0.022706 rpy=0 0 0 -> xyz=0 0.13612 0 rpy=0 0 0
- joint base_weld_arm_right_mount: origin xyz=0.0062926 -0.1505 -0.022706 rpy=0 0 0 -> xyz=0 -0.16488 0 rpy=0 0 0
- joint mount_hand_left_to_arm_left_wrist_mount: origin xyz=-0.028 0 -0.052 rpy=3.1416 0 -1.5708 -> xyz=-0.028 0 -0.0525 rpy=3.1416 0 -1.5708
- joint mount_hand_right_to_arm_right_wrist_mount: origin xyz=-0.028 0 -0.052 rpy=3.1416 0 1.5708 -> xyz=-0.0282 0 -0.0527 rpy=3.1416 0 1.5708

File: packages/linker-robot-assets/src/linker_robot_assets/assets/workstations/a7_lite_o6_dc/workstation.urdf (robot description, URDF)
Before this commit: robot a7_lite_o6_dc, 45 links, 44 joints
Links:
- link base_base_link: mass 8.6616 -> 11.244
Joints:
- joint base_torso_stand: origin xyz=0 0 1.2 rpy=0 0 0 -> xyz=0 0.01438 1.301489 rpy=0 0 0
- joint base_weld_arm_left_mount: origin xyz=0.0062932 0.1505 -0.022706 rpy=0 0 0 -> xyz=0 0.13612 0 rpy=0 0 0
- joint base_weld_arm_right_mount: origin xyz=0.0062926 -0.1505 -0.022706 rpy=0 0 0 -> xyz=0 -0.16488 0 rpy=0 0 0
- joint mount_hand_left_to_arm_left_wrist_mount: origin xyz=-0.028 0 -0.052 rpy=3.1416 0 -1.5708 -> xyz=-0.028 0 -0.0525 rpy=3.1416 0 -1.5708
- joint mount_hand_right_to_arm_right_wrist_mount: origin xyz=-0.028 0 -0.052 rpy=3.1416 0 1.5708 -> xyz=-0.0282 0 -0.0527 rpy=3.1416 0 1.5708
